File: eda/expansion-backplane/expansion-backplane.kicad_pcb (KiCad board)
At the start: 2 copper layers, 235.7 x 78.5 mm, 17 parts, among them J1 OUT1, J10 OUT8, J2 OUT2, J3 PWR, J4 IN, J5 OUT3, J6 OUT4, J7 OUT5, J8 OUT6, J9 OUT7

Commit message: Interim commit
Parts:
- added U1: 74HCT245, Package_DIP:DIP-20_W7.62mm, F.Cu at (264.2, 101.1)
- added U2: 74HCT245, Package_DIP:DIP-20_W7.62mm, F.Cu at (270.5, 112.8)
- added U3: 74HCT245, Package_DIP:DIP-20_W7.62mm, F.Cu at (263.9, 129.0)
- added U4: 74HCT245, Package_DIP:DIP-20_W7.62mm, F.Cu at (270.5, 125.7)
- J2: value OUT2 -> OUT5
- J5: value OUT3 -> OUT2
- J6: value OUT4 -> OUT6
- J7: value OUT5 -> OUT3
- J8: value OUT6 -> OUT7
- J9: value OUT7 -> OUT4
Connections:
- net /IO0 renamed IO0
- net /IO1 renamed IO1
- net /IO2 renamed IO2
- net /IO3 renamed IO3
- net /IO4 renamed IO4
- net /IO5 renamed IO5
- net /IO6 renamed IO6
- net /IO7 renamed IO7
- net /~{IRQ} renamed ~{IRQ}
- net /~{NMI} renamed ~{NMI}
- net /~{RST} renamed ~{RST}
- J1 pad 10: /D3 -> D3
- J1 pad 11: /A4 -> A4
- J1 pad 12: /D4 -> D4
- J1 pad 13: /A5 -> A5
- J1 pad 14: /D5 -> D5
- J1 pad 15: /A6 -> A6
- J1 pad 16: /D6 -> D6
- J1 pad 17: /A7 -> A7
- J1 pad 18: /D7 -> D7
- J1 pad 19: /A8 -> A8
- J1 pad 21: /A9 -> A9
- J1 pad 23: /A10 -> A10
- J1 pad 25: /A11 -> A11
- J1 pad 27: /A12 -> A12
- J1 pad 29: /A13 -> A13
- J1 pad 3: /A0 -> A0
- J1 pad 31: /A14 -> A14
- J1 pad 33: /A15 -> A15
- J1 pad 35: /Clock -> Clock
- J1 pad 37: /R~{W} -> R~{W}
- J1 pad 39: /~{DMA} -> ~{DMA}
- J1 pad 4: /D0 -> D0
- J1 pad 5: /A1 -> A1
- J1 pad 6: /D1 -> D1
- J1 pad 7: /A2 -> A2
- J1 pad 8: /D2 -> D2
- J1 pad 9: /A3 -> A3
- J10 pad 10: /D3 -> D3
- J10 pad 11: /A4 -> A4
- J10 pad 12: /D4 -> D4
- J10 pad 13: /A5 -> A5
- J10 pad 14: /D5 -> D5
- J10 pad 15: /A6 -> A6
- J10 pad 16: /D6 -> D6
- J10 pad 17: /A7 -> A7
- J10 pad 18: /D7 -> D7
- J10 pad 19: /A8 -> A8
- J10 pad 21: /A9 -> A9
- J10 pad 23: /A10 -> A10
- J10 pad 25: /A11 -> A11
- J10 pad 27: /A12 -> A12
- J10 pad 29: /A13 -> A13
- J10 pad 3: /A0 -> A0
- J10 pad 31: /A14 -> A14
- J10 pad 33: /A15 -> A15
- J10 pad 35: /Clock -> Clock
- J10 pad 37: /R~{W} -> R~{W}
- J10 pad 39: /~{DMA} -> ~{DMA}
- J10 pad 4: /D0 -> D0
- J10 pad 5: /A1 -> A1
- J10 pad 6: /D1 -> D1
- J10 pad 7: /A2 -> A2
- J10 pad 8: /D2 -> D2
- J10 pad 9: /A3 -> A3
- J2 pad 10: /D3 -> D3
- J2 pad 11: /A4 -> A4
- J2 pad 12: /D4 -> D4
- J2 pad 13: /A5 -> A5
- J2 pad 14: /D5 -> D5
- J2 pad 15: /A6 -> A6
- J2 pad 16: /D6 -> D6
- J2 pad 17: /A7 -> A7
- J2 pad 18: /D7 -> D7
- J2 pad 19: /A8 -> A8
- J2 pad 21: /A9 -> A9
- J2 pad 23: /A10 -> A10
- J2 pad 25: /A11 -> A11
- J2 pad 27: /A12 -> A12
- J2 pad 29: /A13 -> A13
- J2 pad 3: /A0 -> A0
- J2 pad 31: /A14 -> A14
- J2 pad 33: /A15 -> A15
- J2 pad 35: /Clock -> Clock
- J2 pad 37: /R~{W} -> R~{W}
- J2 pad 39: /~{DMA} -> ~{DMA}
- J2 pad 4: /D0 -> D0
- J2 pad 5: /A1 -> A1
- J2 pad 6: /D1 -> D1
- J2 pad 7: /A2 -> A2
- J2 pad 8: /D2 -> D2
- J2 pad 9: /A3 -> A3
- J4 pad 10: /D3 -> /ID3
- J4 pad 11: /A4 -> /IA4
- J4 pad 12: /D4 -> /ID4
- J4 pad 13: /A5 -> /IA5
- J4 pad 14: /D5 -> /ID5
- J4 pad 15: /A6 -> /IA6
- J4 pad 16: /D6 -> /ID6
- J4 pad 17: /A7 -> /IA7
- J4 pad 18: /D7 -> /ID7
- J4 pad 19: /A8 -> /IA8
- J4 pad 21: /A9 -> /IA9
- J4 pad 23: /A10 -> /IA10
- J4 pad 25: /A11 -> /IA11
- J4 pad 27: /A12 -> /IA12
- J4 pad 29: /A13 -> /IA13
- J4 pad 3: /A0 -> /IA0
- J4 pad 31: /A14 -> /IA14
- J4 pad 33: /A15 -> /IA15
- J4 pad 35: /Clock -> /IClock
- J4 pad 37: /R~{W} -> /IR~{W}
- J4 pad 39: /~{DMA} -> /I~{DMA}
- J4 pad 4: /D0 -> /ID0
- J4 pad 5: /A1 -> /IA1
- J4 pad 6: /D1 -> /ID1
- J4 pad 7: /A2 -> /IA2
- J4 pad 8: /D2 -> /ID2
- J4 pad 9: /A3 -> /IA3
- J5 pad 10: /D3 -> D3
- J5 pad 11: /A4 -> A4
- J5 pad 12: /D4 -> D4
- J5 pad 13: /A5 -> A5
- J5 pad 14: /D5 -> D5
- J5 pad 15: /A6 -> A6
- J5 pad 16: /D6 -> D6
- J5 pad 17: /A7 -> A7
- J5 pad 18: /D7 -> D7
- J5 pad 19: /A8 -> A8
- J5 pad 21: /A9 -> A9
- J5 pad 23: /A10 -> A10
- J5 pad 25: /A11 -> A11
- J5 pad 27: /A12 -> A12
- J5 pad 29: /A13 -> A13
- J5 pad 3: /A0 -> A0
- J5 pad 31: /A14 -> A14
- J5 pad 33: /A15 -> A15
- J5 pad 35: /Clock -> Clock
- J5 pad 37: /R~{W} -> R~{W}
- J5 pad 39: /~{DMA} -> ~{DMA}
- J5 pad 4: /D0 -> D0
- J5 pad 5: /A1 -> A1
- J5 pad 6: /D1 -> D1
- J5 pad 7: /A2 -> A2
- J5 pad 8: /D2 -> D2
- J5 pad 9: /A3 -> A3
- J6 pad 10: /D3 -> D3
- J6 pad 11: /A4 -> A4
- J6 pad 12: /D4 -> D4
- J6 pad 13: /A5 -> A5
- J6 pad 14: /D5 -> D5
- J6 pad 15: /A6 -> A6
- J6 pad 16: /D6 -> D6
- J6 pad 17: /A7 -> A7
- J6 pad 18: /D7 -> D7
- J6 pad 19: /A8 -> A8
- J6 pad 21: /A9 -> A9
- J6 pad 23: /A10 -> A10
- J6 pad 25: /A11 -> A11
- J6 pad 27: /A12 -> A12
- J6 pad 29: /A13 -> A13
- J6 pad 3: /A0 -> A0
- J6 pad 31: /A14 -> A14
- J6 pad 33: /A15 -> A15
- J6 pad 35: /Clock -> Clock
- J6 pad 37: /R~{W} -> R~{W}
- J6 pad 39: /~{DMA} -> ~{DMA}
- J6 pad 4: /D0 -> D0
- J6 pad 5: /A1 -> A1
- J6 pad 6: /D1 -> D1
- J6 pad 7: /A2 -> A2
- J6 pad 8: /D2 -> D2
- J6 pad 9: /A3 -> A3
- J7 pad 10: /D3 -> D3
- J7 pad 11: /A4 -> A4
- J7 pad 12: /D4 -> D4
- J7 pad 13: /A5 -> A5
- J7 pad 14: /D5 -> D5
- J7 pad 15: /A6 -> A6
- J7 pad 16: /D6 -> D6
- J7 pad 17: /A7 -> A7
- J7 pad 18: /D7 -> D7
- J7 pad 19: /A8 -> A8
- J7 pad 21: /A9 -> A9
- J7 pad 23: /A10 -> A10
- J7 pad 25: /A11 -> A11
- J7 pad 27: /A12 -> A12
- J7 pad 29: /A13 -> A13
- J7 pad 3: /A0 -> A0
- J7 pad 31: /A14 -> A14
- J7 pad 33: /A15 -> A15
- J7 pad 35: /Clock -> Clock
- J7 pad 37: /R~{W} -> R~{W}
- J7 pad 39: /~{DMA} -> ~{DMA}
- J7 pad 4: /D0 -> D0
- J7 pad 5: /A1 -> A1
- J7 pad 6: /D1 -> D1
- J7 pad 7: /A2 -> A2
- J7 pad 8: /D2 -> D2
- J7 pad 9: /A3 -> A3
- J8 pad 10: /D3 -> D3
- J8 pad 11: /A4 -> A4
- J8 pad 12: /D4 -> D4
- J8 pad 13: /A5 -> A5
- J8 pad 14: /D5 -> D5
- J8 pad 15: /A6 -> A6
- J8 pad 16: /D6 -> D6
- J8 pad 17: /A7 -> A7
- J8 pad 18: /D7 -> D7
- J8 pad 19: /A8 -> A8
- J8 pad 21: /A9 -> A9
- J8 pad 23: /A10 -> A10
- J8 pad 25: /A11 -> A11
- J8 pad 27: /A12 -> A12
- J8 pad 29: /A13 -> A13
- J8 pad 3: /A0 -> A0
- J8 pad 31: /A14 -> A14
- J8 pad 33: /A15 -> A15
- J8 pad 35: /Clock -> Clock
- J8 pad 37: /R~{W} -> R~{W}
- J8 pad 39: /~{DMA} -> ~{DMA}
- J8 pad 4: /D0 -> D0
- J8 pad 5: /A1 -> A1
- J8 pad 6: /D1 -> D1
- J8 pad 7: /A2 -> A2
- J8 pad 8: /D2 -> D2
- J8 pad 9: /A3 -> A3
- J9 pad 10: /D3 -> D3
- J9 pad 11: /A4 -> A4
- J9 pad 12: /D4 -> D4
- J9 pad 13: /A5 -> A5
- J9 pad 14: /D5 -> D5
- J9 pad 15: /A6 -> A6
- J9 pad 16: /D6 -> D6
- J9 pad 17: /A7 -> A7
- J9 pad 18: /D7 -> D7
- J9 pad 19: /A8 -> A8
- J9 pad 21: /A9 -> A9
- J9 pad 23: /A10 -> A10
- J9 pad 25: /A11 -> A11
- J9 pad 27: /A12 -> A12
- J9 pad 29: /A13 -> A13
- J9 pad 3: /A0 -> A0
- J9 pad 31: /A14 -> A14
- J9 pad 33: /A15 -> A15
- J9 pad 35: /Clock -> Clock
- J9 pad 37: /R~{W} -> R~{W}
- J9 pad 39: /~{DMA} -> ~{DMA}
- J9 pad 4: /D0 -> D0
- J9 pad 5: /A1 -> A1
- J9 pad 6: /D1 -> D1
- J9 pad 7: /A2 -> A2
- J9 pad 8: /D2 -> D2
- J9 pad 9: /A3 -> A3
Routing:
- net A7: track 0.00 -> 210.8 mm
- net A6: track 0.00 -> 210.7 mm
- net A5: track 0.00 -> 209.9 mm
- net A4: track 0.00 -> 209.8 mm
- net A3: track 0.00 -> 209.0 mm
- net A2: track 0.00 -> 208.5 mm
- net A1: track 0.00 -> 206.5 mm
- net A0: track 0.00 -> 204.2 mm
- net D4: track 0.00 -> 174.8 mm
- net D2: track 0.00 -> 174.7 mm
- net D6: track 0.00 -> 174.7 mm
- net D7: track 0.00 -> 174.7 mm
- net D1: track 0.00 -> 174.7 mm
- net D0: track 0.00 -> 174.6 mm
- net D5: track 0.00 -> 174.5 mm
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
Commit message: Update cap footprint
Parts:
- added C2: 100nf, Capacitor_THT:C_Rect_L7.2mm_W3.5mm_P5.00mm_FKS2_FKP2_MKS2_MKP2, F.Cu at (269.3, 129.5)
- added C3: 100nf, Capacitor_THT:C_Rect_L7.2mm_W3.5mm_P5.00mm_FKS2_FKP2_MKS2_MKP2, F.Cu at (302.3, 104.1)
- added C4: 100nf, Capacitor_THT:C_Rect_L7.2mm_W3.5mm_P5.00mm_FKS2_FKP2_MKS2_MKP2, F.Cu at (271.8, 81.3)
- added C5: 100nf, Capacitor_THT:C_Rect_L7.2mm_W3.5mm_P5.00mm_FKS2_FKP2_MKS2_MKP2, F.Cu at (251.5, 132.0)
