File: eda/expansion-backplane/expansion-backplane.kicad_sch (KiCad schematic)
At the start: 15 parts, among them J1 IN, J2 OUT3, J2 OUT4, J2 OUT7, J2 OUT8, J3 OUT2, J3 OUT6, J4 OUT1, J4 OUT5, J5 PWR

Commit message: Interim commit
Parts:
- removed J2: OUT3, Connector_PinSocket_2.54mm:PinSocket_2x20_P2.54mm_Vertical, symbol Connector_Generic:Conn_02x20_Odd_Even
- removed J2: OUT7, Connector_PinSocket_2.54mm:PinSocket_2x20_P2.54mm_Vertical, symbol Connector_Generic:Conn_02x20_Odd_Even
- removed J2: OUT4, Connector_PinSocket_2.54mm:PinSocket_2x20_P2.54mm_Vertical, symbol Connector_Generic:Conn_02x20_Odd_Even
- removed J2: OUT8, Connector_PinSocket_2.54mm:PinSocket_2x20_P2.54mm_Vertical, symbol Connector_Generic:Conn_02x20_Odd_Even
- removed J3: OUT2, Connector_PinSocket_2.54mm:PinSocket_2x20_P2.54mm_Vertical, symbol Connector_Generic:Conn_02x20_Odd_Even
- removed J3: OUT6, Connector_PinSocket_2.54mm:PinSocket_2x20_P2.54mm_Vertical, symbol Connector_Generic:Conn_02x20_Odd_Even
- removed J4: OUT5, Connector_PinSocket_2.54mm:PinSocket_2x20_P2.54mm_Vertical, symbol Connector_Generic:Conn_02x20_Odd_Even
- removed J4: OUT1, Connector_PinSocket_2.54mm:PinSocket_2x20_P2.54mm_Vertical, symbol Connector_Generic:Conn_02x20_Odd_Even
- added C2, C3, C4, C5: 100nf, symbol Device:C
- added U1, U2, U3, U4: 74HCT245, Package_DIP:DIP-20_W7.62mm, symbol 74xx:74LS245
Connections:
- net A0: now also U2.18 (B0); no longer J1.3 (Pin_3)
- net A1: now also U2.17 (B1); no longer J1.5 (Pin_5)
- net A10: now also U3.13 (B5); no longer J1.23 (Pin_23)
- net A11: now also U3.14 (B4); no longer J1.25 (Pin_25)
- net A12: now also U3.15 (B3); no longer J1.27 (Pin_27)
- net A13: now also U3.16 (B2); no longer J1.29 (Pin_29)
- net A14: now also U3.17 (B1); no longer J1.31 (Pin_31)
- net A15: now also U3.18 (B0); no longer J1.33 (Pin_33)
- net A2: now also U2.16 (B2); no longer J1.7 (Pin_7)
- net A3: now also U2.15 (B3); no longer J1.9 (Pin_9)
- net A4: now also U2.14 (B4); no longer J1.11 (Pin_11)
- net A5: now also U2.13 (B5); no longer J1.13 (Pin_13)
- net A6: now also U2.12 (B6); no longer J1.15 (Pin_15)
- net A7: now also U2.11 (B7); no longer J1.17 (Pin_17)
- net A8: now also U3.11 (B7); no longer J1.19 (Pin_19)
- net A9: now also U3.12 (B6); no longer J1.21 (Pin_21)
- net Clock: now also U4.18 (B0); no longer J1.35 (Pin_35)
- net D0: now also U1.9 (A7); no longer J1.4 (Pin_4)
- net D1: now also U1.8 (A6); no longer J1.6 (Pin_6)
- net D2: now also U1.7 (A5); no longer J1.8 (Pin_8)
- net D3: now also U1.6 (A4); no longer J1.10 (Pin_10)
- net D4: now also U1.5 (A3); no longer J1.12 (Pin_12)
- net D5: now also U1.4 (A2); no longer J1.14 (Pin_14)
- net D6: now also U1.3 (A1); no longer J1.16 (Pin_16)
- net D7: now also U1.2 (A0); no longer J1.18 (Pin_18)
- net GND: now also C2.2, C3.2, C4.2, C5.2, U1.10 (GND), U1.19 (CE), U2.10 (GND), U2.19 (CE), U3.10 (GND), U3.19 (CE), U4.10 (GND), U4.19 (CE)
- net R~{W}: now also U4.17 (B1); no longer J1.37 (Pin_37)
- net VCC: now also C2.1, C3.1, C4.1, C5.1, U1.20 (VCC), U2.1 (A->B), U2.20 (VCC), U3.1 (A->B), U3.20 (VCC), U4.1 (A->B), U4.20 (VCC), U4.5 (A3), U4.6 (A4), U4.7 (A5), U4.8 (A6), U4.9 (A7)
- net ~{DMA}: now also U4.16 (B2); no longer J1.39 (Pin_39)
- new net IA0: J1.3 (Pin_3), U2.2 (A0)
- new net IA1: J1.5 (Pin_5), U2.3 (A1)
- new net IA10: J1.23 (Pin_23), U3.7 (A5)
- new net IA11: J1.25 (Pin_25), U3.6 (A4)
- new net IA12: J1.27 (Pin_27), U3.5 (A3)
- new net IA13: J1.29 (Pin_29), U3.4 (A2)
- new net IA14: J1.31 (Pin_31), U3.3 (A1)
- new net IA15: J1.33 (Pin_33), U3.2 (A0)
- new net IA2: J1.7 (Pin_7), U2.4 (A2)
- new net IA3: J1.9 (Pin_9), U2.5 (A3)
- new net IA4: J1.11 (Pin_11), U2.6 (A4)
- new net IA5: J1.13 (Pin_13), U2.7 (A5)
- new net IA6: J1.15 (Pin_15), U2.8 (A6)
- new net IA7: J1.17 (Pin_17), U2.9 (A7)
- new net IA8: J1.19 (Pin_19), U3.9 (A7)
- new net IA9: J1.21 (Pin_21), U3.8 (A6)
- new net IClock: J1.35 (Pin_35), U4.2 (A0)
- new net ID0: J1.4 (Pin_4), U1.11 (B7)
- new net ID1: J1.6 (Pin_6), U1.12 (B6)
- new net ID2: J1.8 (Pin_8), U1.13 (B5)
- new net ID3: J1.10 (Pin_10), U1.14 (B4)
- new net ID4: J1.12 (Pin_12), U1.15 (B3)
- new net ID5: J1.14 (Pin_14), U1.16 (B2)
- new net ID6: J1.16 (Pin_16), U1.17 (B1)
- new net ID7: J1.18 (Pin_18), U1.18 (B0)
- new net IR~{W}: J1.37 (Pin_37), U1.1 (A->B), U4.3 (A1)
- new net I~{DMA}: J1.39 (Pin_39), U4.4 (A2)
Other:
- added sheet Outputs (outputs.kicad_sch)
- moved on the sheet: H1, H2, H3, H4

Commit message: Update cap footprint
Parts:
- C2, C3, C4, C5: footprint (none) -> Capacitor_THT:C_Rect_L7.2mm_W3.5mm_P5.00mm_FKS2_FKP2_MKS2_MKP2
