File: eda/lcd-interface/lcd-interface.kicad_pcb (KiCad board)
At the start: 2 copper layers, 140.2 x 81.3 mm, 20 parts, among them J1 Conn_02x25_Odd_Even, U1 W65C22SxP, U2 LCD-016N002L

Commit message: Normalize cap size
Parts:
- C2, C3: footprint Capacitor_THT:C_Disc_D3.4mm_W2.1mm_P2.50mm -> Capacitor_THT:C_Disc_D3.8mm_W2.6mm_P2.50mm
- R1: value Backlight (R or Jumper) -> LED-R (DNP)
- renumbered C1 to C18, J1 to J2
