File: eda/main-board/main-board.kicad_pcb (KiCad board)
At the start: 2 copper layers, 64 parts, among them J1 RomHighSel, J2 Membank block, J3 Expansion, J4 $1-3 latch, J5 PWR, J6 CS_leds, U1 W65C02SxP, U10 74HCT00, U11 74HCT32, U12 74HCT32, U13 74HCT138, U14 74LHCT157, U15 74LHCT157, U16 74HCT273, U2 NA555P, U3 28C256, U4 AS6C4008-55PCN, U5 74HCT138, U6 74HCT32, U7 74HCT08, U8 74HCT30, U9 74HCT139, X1 4Mhz

Commit message: Work on main board eda, interim
Parts:
- moved U13 74.9 mm to (274.8, 134.1)
- moved C8 69.6 mm to (281.2, 130.4), turned to 180 degrees
- moved U4 48.3 mm to (75.2, 149.9), turned to 180 degrees
- moved U3 39.1 mm to (109.2, 146.3), turned to 180 degrees
- moved U1 18.2 mm to (33.5, 101.9)
- moved C5 7.62 mm to (266.8, 100.1)
- moved J3 7.62 mm to (267.2, 108.7)
- moved X1 0.69 mm to (240.5, 126.4)
Connections:
- U13 pad 10: unconnected-(U13-O5-Pad10) -> /IO Address Decode/IoSelect5
- U13 pad 11: unconnected-(U13-O4-Pad11) -> /IO Address Decode/IoSelect4
- U13 pad 12: unconnected-(U13-O3-Pad12) -> /IO Address Decode/IoSelect3
- U13 pad 13: unconnected-(U13-O2-Pad13) -> /IO Address Decode/IoSelect2
- U13 pad 14: unconnected-(U13-O1-Pad14) -> /IO Address Decode/IoSelect1
- U13 pad 15: unconnected-(U13-O0-Pad15) -> /IO Address Decode/IoSelect0
- U13 pad 7: unconnected-(U13-O7-Pad7) -> /IO Address Decode/IoSelect7
- U13 pad 9: unconnected-(U13-O6-Pad9) -> /IO Address Decode/IoSelect6
Routing:
- net GND: track 0.00 -> 30.3 mm
- net /IO Address Decode/IoSelect5: track 0.00 -> 14.8 mm
- net /IO Address Decode/IoSelect4: track 0.00 -> 14.8 mm
- net /IO Address Decode/IoSelect2: track 0.00 -> 14.8 mm
- net /IO Address Decode/IoSelect1: track 0.00 -> 14.8 mm
- net /IO Address Decode/IoSelect6: track 0.00 -> 14.8 mm
- net /IO Address Decode/IoSelect3: track 0.00 -> 14.8 mm
- net /IO Address Decode/IoSelect0: track 0.00 -> 14.8 mm
- net /IO Address Decode/IoSelect7: track 0.00 -> 5.08 mm
- net VCC: track 0.00 -> 4.24 mm

Commit message: Update eda
Routing:
- net /Address decode/~{Io1Cs}: track 0.00 -> 2.54 mm
Changed lines of the file:
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@@
   (segment (start 269.748 146.812) (end 270.873 147.937) (width 0.25) (layer "F.Cu") (net 63))
   (segment (start 274.828 149.352) (end 269.748 149.352) (width 0.25) (layer "F.Cu") (net 64))
+  (segment (start 274.828 144.272) (end 274.828 141.732) (width 0.25) (layer "B.Cu") (net 77))
 )

Commit message: Add expansion backplane
Parts:
- removed U11: 74HCT32, Package_DIP:DIP-14_W7.62mm
- added H1: MountingHole, MountingHole:MountingHole_2.1mm, F.Cu at (63.2, 44.2)
- added H2: MountingHole, MountingHole:MountingHole_2.1mm, F.Cu at (204.3, 44.2)
- added H3: MountingHole, MountingHole:MountingHole_2.1mm, F.Cu at (63.2, 135.5)
- added H4: MountingHole, MountingHole:MountingHole_2.1mm, F.Cu at (204.2, 135.4)
- moved J4 197.8 mm to (64.5, 70.6)
- moved R3 162.7 mm to (97.7, 50.4)
- moved J1 161.3 mm to (109.8, 44.7), turned to -90 degrees
- moved R4 148.6 mm to (73.2, 106.4), turned to 90 degrees
- moved X1 145.4 mm to (102.0, 82.4)
- moved J6 142.5 mm to (64.6, 50.9)
- moved U1 135.8 mm to (166.3, 73.2), turned to -90 degrees
- moved R5 125.8 mm to (90.3, 79.2), turned to 180 degrees
- moved U9 122.3 mm to (67.9, 116.0)
- moved C13 122.3 mm to (74.0, 112.5)
- moved U12 119.7 mm to (120.0, 98.3), turned to -90 degrees
- moved C8 118.7 mm to (199.1, 44.7)
- moved U13 118.7 mm to (192.7, 48.4)
- moved U4 114.1 mm to (187.6, 129.8)
- moved C18 97.9 mm to (182.7, 135.0)
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Routing:
- net /IO Address Decode/IoSelect5: track 14.8 -> 0.00 mm
- net /IO Address Decode/IoSelect4: track 14.8 -> 0.00 mm
- net /IO Address Decode/IoSelect2: track 14.8 -> 0.00 mm
- net /IO Address Decode/IoSelect1: track 14.8 -> 0.00 mm
- net /IO Address Decode/IoSelect6: track 14.8 -> 0.00 mm
- net /IO Address Decode/IoSelect3: track 14.8 -> 0.00 mm
- net /IO Address Decode/IoSelect0: track 14.8 -> 0.00 mm
- net /IO Address Decode/IoSelect7: track 5.08 -> 0.00 mm
Other:
- board outline added: 146.3 x 96.5 mm

Commit message: EDA work for new expansion header
Parts:
- removed the C6 at (90.4, 47.1)
- added C20: 100n, Capacitor_THT:C_Disc_D6.0mm_W2.5mm_P5.00mm, F.Cu at (225.2, 68.5)
- added C21: 100n, Capacitor_THT:C_Disc_D6.0mm_W2.5mm_P5.00mm, F.Cu at (241.9, 61.7)
- added C22: 100n, Capacitor_THT:C_Disc_D6.0mm_W2.5mm_P5.00mm, F.Cu at (242.2, 93.8)
- added C23: 100n, Capacitor_THT:C_Disc_D6.0mm_W2.5mm_P5.00mm, F.Cu at (217.4, 94.2)
- added J7: Expansion, Connector_PinHeader_2.54mm:PinHeader_2x25_P2.54mm_Vertical, F.Cu at (254.8, 64.0)
- added R9: 10k, Resistor_THT:R_Axial_DIN0207_L6.3mm_D2.5mm_P7.62mm_Horizontal, F.Cu at (262.5, 129.6)
- added U11: 74HCT245, Package_DIP:DIP-20_W7.62mm, F.Cu at (223.7, 72.1)
- added U17: 74HCT541, Package_DIP:DIP-20_W7.62mm, F.Cu at (240.7, 65.6)
- added U18: 74HCT541, Package_DIP:DIP-20_W7.62mm, F.Cu at (240.8, 97.6)
- added U20: 74HCT541, Package_DIP:DIP-20_W7.62mm, F.Cu at (211.2, 98.0)
- C6: value 100n -> 3u; footprint Capacitor_THT:C_Disc_D6.0mm_W2.5mm_P5.00mm -> Capacitor_THT:CP_Radial_D8.0mm_P3.50mm
- J3: value Expansion -> ResetSwitch; footprint Connector_PinHeader_2.54mm:PinHeader_2x20_P2.54mm_Vertical -> Connector_PinHeader_2.54mm:PinHeader_1x02_P2.54mm_Vertical
- moved H3 221.2 mm to (264.4, 43.4)
- moved J5 175.1 mm to (253.7, 47.0)
- moved H2 148.4 mm to (55.9, 43.2)
- moved C2 147.0 mm to (224.6, 47.5)
- moved R1 145.5 mm to (215.5, 64.2)
- moved U2 145.5 mm to (232.6, 52.2)
- moved C3 145.4 mm to (230.1, 46.9)
- moved C1 145.3 mm to (217.9, 60.1)
- moved C6 135.1 mm to (262.4, 53.9), turned to 0 degrees
- moved R2 121.7 mm to (238.2, 59.8), turned to 90 degrees
- moved X1 112.0 mm to (209.8, 52.2), turned to 90 degrees
- moved R5 109.7 mm to (196.1, 50.6), turned to -90 degrees
- moved J2 106.8 mm to (88.1, 44.6), turned to 90 degrees
- moved H1 93.2 mm to (55.9, 137.2)
- moved R4 91.9 mm to (164.9, 111.1), turned to -90 degrees
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Connections:
- net Net-(J2-Pin_2) renamed /Memory banking/LA13
- net Net-(J2-Pin_3) renamed /Memory banking/LA14
- net Net-(J2-Pin_4) renamed /Memory banking/LA15
- net Net-(J2-Pin_5) renamed /Memory banking/LA17
- net Net-(J2-Pin_6) renamed /Memory banking/LA18
- net Net-(U5-O6) renamed /Address decode/C000
- net Net-(U5-O7) renamed /Address decode/E000
- D1 pad 2: /Address decode/A12 -> /A12
- D10 pad 2: /Address decode/A3 -> /A3
- D11 pad 2: /Address decode/A2 -> /A2
- D2 pad 2: /Address decode/A11 -> /A11
- D3 pad 2: /Address decode/A10 -> /A10
- D4 pad 2: /Address decode/A9 -> /A9
- D5 pad 2: /Address decode/A8 -> /A8
- D6 pad 2: /Address decode/A7 -> /A7
- D7 pad 2: /Address decode/A6 -> /A6
- D8 pad 2: /Address decode/A5 -> /A5
- D9 pad 2: /Address decode/A4 -> /A4
- J3 pad 1: VCC -> Net-(J3-Pin_1)
- R5 pad 2: /Memory banking/~{Reset} -> /Expansion/~{RST}
- R6 pad 2: Net-(J3-Pin_40) -> /Expansion/e/~{NMI}
- R7 pad 2: Net-(J3-Pin_38) -> Net-(J3-Pin_1)
- R8 pad 2: Net-(J3-Pin_39) -> /Expansion/e/~{IRQ}
- U1 pad 2: Net-(J3-Pin_39) -> /Expansion/~{DMA}
- U1 pad 36: Net-(J3-Pin_39) -> /Expansion/~{DMA}
- U1 pad 37: Clock -> /RawClock
- U1 pad 39: unconnected-(U1-ϕ2-Pad39) -> Clock
- U1 pad 4: Net-(J3-Pin_40) -> /Expansion/~{IRQ}
- U1 pad 40: /Memory banking/~{Reset} -> /Expansion/~{RST}
- U1 pad 6: Net-(J3-Pin_38) -> /Expansion/~{NMI}
- U10 pad 1: /Address decode/A11 -> /A11
- U10 pad 11: /Memory banking/~{Reset} -> /Expansion/~{RST}
- U10 pad 2: /Address decode/A12 -> /A12
- U12 pad 10: (no net) -> GND
- U12 pad 11: (no net) -> unconnected-(U12-Pad11)
- U12 pad 12: (no net) -> GND
- U12 pad 13: (no net) -> GND
- U12 pad 14: (no net) -> VCC
- U12 pad 4: (no net) -> GND
- U12 pad 5: (no net) -> GND
- U12 pad 6: (no net) -> unconnected-(U12-Pad6)
- U12 pad 7: (no net) -> GND
- U12 pad 8: (no net) -> unconnected-(U12-Pad8)
- U12 pad 9: (no net) -> GND
- U13 pad 1: /Address decode/A6 -> /A6
- U13 pad 10: /IO Address Decode/IoSelect5 -> /Expansion/IoSelect5
- U13 pad 11: /IO Address Decode/IoSelect4 -> /Expansion/IoSelect4
- U13 pad 12: /IO Address Decode/IoSelect3 -> /Expansion/IoSelect3
- U13 pad 13: /IO Address Decode/IoSelect2 -> /Expansion/IoSelect2
- U13 pad 14: /IO Address Decode/IoSelect1 -> /Expansion/IoSelect1
- U13 pad 15: /IO Address Decode/IoSelect0 -> /Expansion/IoSelect0
- U13 pad 2: /Address decode/A7 -> /A7
- U13 pad 3: /Address decode/A8 -> /A8
- U13 pad 7: /IO Address Decode/IoSelect7 -> /Expansion/IoSelect7
- U13 pad 9: /IO Address Decode/IoSelect6 -> /Expansion/IoSelect6
- U14 pad 10: /Address decode/A15 -> /A15
- U14 pad 3: /Address decode/A13 -> /A13
- U14 pad 6: /Address decode/A14 -> /A14
- U16 pad 1: /Memory banking/~{Reset} -> /Expansion/~{RST}
- U16 pad 3: /D0 -> /D1
- U16 pad 4: /D1 -> /D0
- U2 pad 4: VCC -> Net-(J3-Pin_1)
- U3 pad 10: /Address decode/A0 -> /A0
- U3 pad 2: /Address decode/A12 -> /A12
- U3 pad 21: /Address decode/A10 -> /A10
- U3 pad 23: /Address decode/A11 -> /A11
- U3 pad 24: /Address decode/A9 -> /A9
- U3 pad 25: /Address decode/A8 -> /A8
- U3 pad 26: /Address decode/A13 -> /A13
- U3 pad 3: /Address decode/A7 -> /A7
- U3 pad 4: /Address decode/A6 -> /A6
- U3 pad 5: /Address decode/A5 -> /A5
- U3 pad 6: /Address decode/A4 -> /A4
- U3 pad 7: /Address decode/A3 -> /A3
- U3 pad 8: /Address decode/A2 -> /A2
- U3 pad 9: /Address decode/A1 -> /A1
- U4 pad 10: /Address decode/A2 -> /A2
- U4 pad 11: /Address decode/A1 -> /A1
- U4 pad 12: /Address decode/A0 -> /A0
- U4 pad 23: /Address decode/A10 -> /A10
- U4 pad 25: /Address decode/A11 -> /A11
- U4 pad 26: /Address decode/A9 -> /A9
- U4 pad 27: /Address decode/A8 -> /A8
- U4 pad 4: /Address decode/A12 -> /A12
- U4 pad 5: /Address decode/A7 -> /A7
- U4 pad 6: /Address decode/A6 -> /A6
- U4 pad 7: /Address decode/A5 -> /A5
- U4 pad 8: /Address decode/A4 -> /A4
- U4 pad 9: /Address decode/A3 -> /A3
- U5 pad 1: /Address decode/A13 -> /A13
- U5 pad 2: /Address decode/A14 -> /A14
- U5 pad 3: /Address decode/A15 -> /A15
- U9 pad 13: /Address decode/A0 -> /A0
- U9 pad 14: /Address decode/A1 -> /A1
- U9 pad 2: /Address decode/A10 -> /A10
- U9 pad 3: /Address decode/A9 -> /A9
- X1 pad 5: Clock -> /RawClock
Routing:
- net VCC: track 4.24 -> 747.2 mm, vias 0 -> 8
- net /A13: track 0.00 -> 270.7 mm, vias 0 -> 7
- net /A11: track 0.00 -> 240.9 mm, vias 0 -> 3
- net /A5: track 0.00 -> 230.7 mm, vias 0 -> 5
- net /A6: track 0.00 -> 217.2 mm, vias 0 -> 4
- net /A10: track 0.00 -> 211.9 mm, vias 0 -> 4
- net /A2: track 0.00 -> 206.2 mm, vias 0 -> 2
- net /A7: track 0.00 -> 202.6 mm, vias 0 -> 4
- net /A8: track 0.00 -> 196.3 mm, vias 0 -> 5
- net /A15: track 0.00 -> 194.5 mm, vias 0 -> 4
- net /A4: track 0.00 -> 190.4 mm, vias 0 -> 2
- net /A9: track 0.00 -> 189.5 mm, vias 0 -> 4
- net /A14: track 0.00 -> 185.8 mm, vias 0 -> 5
- net /D4: track 0.00 -> 184.7 mm, vias 0 -> 2
- net /D3: track 0.00 -> 181.9 mm, vias 0 -> 2
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- added copper zone on B.Cu, net GND
Other:
- board size 146.3 x 96.5 mm -> 217.2 x 104.1 mm
- board text added: "Project WRASS - Main Board v2.0 Niklas Hedlund, 2024"

Commit message: Branch of uart to v1
Parts:
- added D14: LED, LED_THT:LED_D3.0mm, F.Cu at (225.4, 43.8)
- added H5: MountingHole_Pad, MountingHole:MountingHole_2.5mm_Pad_Via, F.Cu at (172.5, 44.0)
- added H6: MountingHole_Pad, MountingHole:MountingHole_2.5mm_Pad_Via, F.Cu at (172.7, 135.0)
- added R10: 1k, Resistor_THT:R_Axial_DIN0207_L6.3mm_D2.5mm_P7.62mm_Horizontal, F.Cu at (229.2, 43.2)
- H1, H2, H3, H4: value MountingHole -> MountingHole_Pad; footprint MountingHole:MountingHole_2.1mm -> MountingHole:MountingHole_2.5mm_Pad_Via
- moved H1 94.2 mm to (42.4, 43.9)
- moved H2 92.7 mm to (42.4, 134.9)
- moved R3 22.6 mm to (158.1, 43.2)
- moved J1 12.8 mm to (165.4, 43.2)
- moved C6 11.8 mm to (251.0, 57.1)
- moved C5 7.42 mm to (261.1, 57.4)
- moved R1 3.80 mm to (213.4, 67.3)
- moved R2 3.78 mm to (237.5, 63.5)
- moved U2 3.67 mm to (232.6, 55.9)
- moved C1 3.49 mm to (217.2, 63.5)
- moved C2 3.31 mm to (224.8, 50.8)
- moved R7 3.25 mm to (217.2, 47.6)
- moved C3 2.05 mm to (230.5, 48.9)
- moved J2 1.63 mm to (88.1, 46.2)
- moved J3 1.13 mm to (240.7, 45.7)
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Routing:
- net VCC: track 747.2 -> 7.50 mm, vias 8 -> 0
- net Net-(U10-Pad3): track 0.00 -> 181.6 mm, vias 0 -> 4
- net /Address decode/~{RomCs}: track 12.2 -> 162.0 mm, vias 0 -> 2
- net /Address decode/~{Io1Cs}: track 34.4 -> 180.9 mm, vias 0 -> 2
- net /Address decode/R~{W}: track 48.1 -> 187.7 mm, vias 0 -> 4
- net /Expansion/~{RST}: track 116.3 -> 225.1 mm, vias 1 -> 2
- net /A1: track 99.7 -> 208.0 mm, vias 0 -> 5
- net /A0: track 100.0 -> 208.3 mm, vias 0 -> 5
- net ~{8000}: track 14.2 -> 107.2 mm, vias 0 -> 2
- net Net-(J7-Pin_41): track 0.00 -> 86.6 mm, vias 0 -> 3
- net /Address decode/~{RamOe}: track 38.1 -> 122.8 mm, vias 1 -> 3
- net /Address decode/~{RamCs}: track 38.3 -> 116.8 mm, vias 1 -> 4
- net Net-(J7-Pin_43): track 0.00 -> 77.8 mm, vias 0 -> 3
- net Net-(J7-Pin_39): track 18.3 -> 94.9 mm, vias 0 -> 2
- net Net-(J1-Pin_2): track 6.91 -> 61.2 mm, vias 0 -> 2
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- added copper zone on In2.Cu, net GND
- added copper zone on In1.Cu, net VCC
Other:
- board size 217.2 x 104.1 mm -> 230 x 100 mm
- copper layers 2 -> 4
- board text added: "$1"
- board text added: "$2"
- board text added: "$3"
- board text added: "GND"
- board text added: "IO1"
- board text added: "IO2"
- board text added: "LA13"
- board text added: "LA14"
- board text added: "LA15"
- board text added: "LA17"
- board text added: "LA18"
- board text added: "RAM"
- board text added: "RO1"
- board text added: "RO2"
- board text added: "VCC"

Commit message: Generate step files and start on gpu for new board layout
Routing:
- net /D2: track 181.5 -> 134.5 mm, vias 3 -> 1
- net /A11: track 281.6 -> 264.4 mm
- net VCC: track 7.50 -> 4.84 mm
- net Net-(J1-Pin_2): track 61.2 -> 60.2 mm
- net /A8: track 196.3 -> 195.3 mm
- net Net-(J7-Pin_41): track 86.6 -> 86.1 mm
- net /Address decode/~{RamCs}: track 116.8 -> 116.2 mm
- net Net-(U10-Pad3): vias 4 -> 3

Commit message: Normalize cap size
Parts:
- C10, C11, C12, C13, C14, C15, C16, C17, C18, C19, C20, C21, C22, C23, C3, C4, C7, C8, C9: footprint Capacitor_THT:C_Disc_D6.0mm_W2.5mm_P5.00mm -> Capacitor_THT:C_Disc_D3.8mm_W2.6mm_P2.50mm
