File: eda/main-board/address-decode.kicad_sch (KiCad schematic)
At the start: 30 parts, among them J6 CS_leds, U10 74HCT00, U11 74HCT32, U12 74HCT32, U5 74HCT138, U6 74HCT32, U7 74HCT08, U8 74HCT30, U9 74HCT139

Commit message: Work on main board eda, interim
Other:
- moved on the sheet: U10B
Changed lines of the file:
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@@
   (junction (at 87.63 190.5) (diameter 0) (color 0 0 0 0)
   )
+  (junction (at 257.81 113.03) (diameter 0) (color 0 0 0 0)
+  )
   (junction (at 257.81 138.43) (diameter 0) (color 0 0 0 0)
   )
@@
   )
   (junction (at 162.56 161.29) (diameter 0) (color 0 0 0 0)
-  )
-  (junction (at 257.81 123.19) (diameter 0) (color 0 0 0 0)
   )
   (junction (at 60.96 64.77) (diameter 0) (color 0 0 0 0)
@@
   (no_connect (at 85.09 90.17))
   (no_connect (at 273.05 130.81))
-  (no_connect (at 273.05 120.65))
+  (no_connect (at 273.05 110.49))
   (no_connect (at 73.66 39.37))
   (no_connect (at 273.05 140.97))
@@
     (stroke (width 0) (type default))
   )
-  (wire (pts (xy 257.81 123.19) (xy 257.81 128.27))
+  (wire (pts (xy 257.81 113.03) (xy 257.81 128.27))
     (stroke (width 0) (type default))
   )
@@
     (stroke (width 0) (type default))
   )
-  (wire (pts (xy 257.81 118.11) (xy 257.81 123.19))
+  (wire (pts (xy 257.81 107.95) (xy 257.81 113.03))
     (stroke (width 0) (type default))
   )
@@
     (stroke (width 0) (type default))
   )
-  (label "A11" (at 24.13 110.49 0)
-    (effects (font (size 1.27 1.27)) (justify left bottom))
-  )
-  (label "A12" (at 22.86 82.55 0)
-    (effects (font (size 1.27 1.27)) (justify left bottom))
-  )
-  (label "A2" (at 24.13 144.78 0)
-    (effects (font (size 1.27 1.27)) (justify left bottom))
-  )
-  (label "A3" (at 24.13 140.97 0)
-    (effects (font (size 1.27 1.27)) (justify left bottom))
-  )
-  (label "A8" (at 24.13 121.92 0)
-    (effects (font (size 1.27 1.27)) (justify left bottom))
-  )
-  (label "A0" (at 57.15 110.49 0)
-    (effects (font (size 1.27 1.27)) (justify left bottom))
-  )
-  (label "A11" (at 22.86 77.47 0)
-    (effects (font (size 1.27 1.27)) (justify left bottom))
-  )
-  (label "A7" (at 24.13 125.73 0)
-    (effects (font (size 1.27 1.27)) (justify left bottom))
-  )
-  (label "A5" (at 24.13 133.35 0)
-    (effects (font (size 1.27 1.27)) (justify left bottom))
-  )
-  (label "A12" (at 24.13 106.68 0)
-    (effects (font (size 1.27 1.27)) (justify left bottom))
-  )
-  (label "A10" (at 57.15 87.63 0)
-    (effects (font (size 1.27 1.27)) (justify left bottom))
-  )
-  (label "A9" (at 57.15 85.09 0)
-    (effects (font (size 1.27 1.27)) (justify left bottom))
-  )
-  (label "A6" (at 24.13 129.54 0)
-    (effects (font (size 1.27 1.27)) (justify left bottom))
-  )
-  (label "A13" (at 40.64 36.83 0)
-    (effects (font (size 1.27 1.27)) (justify left bottom))
-  )
-  (label "A9" (at 24.13 118.11 0)
-    (effects (font (size 1.27 1.27)) (justify left bottom))
-  )
-  (label "A4" (at 24.13 137.16 0)
-    (effects (font (size 1.27 1.27)) (justify left bottom))
-  )
-  (label "A15" (at 40.64 41.91 0)
-    (effects (font (size 1.27 1.27)) (justify left bottom))
-  )
-  (label "A14" (at 40.64 39.37 0)
-    (effects (font (size 1.27 1.27)) (justify left bottom))
-  )
-  (label "A1" (at 57.15 113.03 0)
-    (effects (font (size 1.27 1.27)) (justify left bottom))
-  )
-  (label "A10" (at 24.13 114.3 0)
+  (label "A11" (at 24.13 110.49 0) (fields_autoplaced)
+    (effects (font (size 1.27 1.27)) (justify left bottom))
+  )
+  (label "A12" (at 22.86 82.55 0) (fields_autoplaced)
+    (effects (font (size 1.27 1.27)) (justify left bottom))
+  )
+  (label "A2" (at 24.13 144.78 0) (fields_autoplaced)
+    (effects (font (size 1.27 1.27)) (justify left bottom))
+  )
+  (label "A3" (at 24.13 140.97 0) (fields_autoplaced)
+    (effects (font (size 1.27 1.27)) (justify left bottom))
+  )
+  (label "A8" (at 24.13 121.92 0) (fields_autoplaced)
+    (effects (font (size 1.27 1.27)) (justify left bottom))
+  )
+  (label "A0" (at 57.15 110.49 0) (fields_autoplaced)
+    (effects (font (size 1.27 1.27)) (justify left bottom))
+  )
+  (label "A11" (at 22.86 77.47 0) (fields_autoplaced)
+    (effects (font (size 1.27 1.27)) (justify left bottom))
+  )
+  (label "A7" (at 24.13 125.73 0) (fields_autoplaced)
+    (effects (font (size 1.27 1.27)) (justify left bottom))
+  )
+  (label "A5" (at 24.13 133.35 0) (fields_autoplaced)
+    (effects (font (size 1.27 1.27)) (justify left bottom))
+  )
+  (label "A12" (at 24.13 106.68 0) (fields_autoplaced)
+    (effects (font (size 1.27 1.27)) (justify left bottom))
+  )
+  (label "A10" (at 57.15 87.63 0) (fields_autoplaced)
+    (effects (font (size 1.27 1.27)) (justify left bottom))
+  )
+  (label "A9" (at 57.15 85.09 0) (fields_autoplaced)
+    (effects (font (size 1.27 1.27)) (justify left bottom))
+  )
+  (label "A6" (at 24.13 129.54 0) (fields_autoplaced)
+    (effects (font (size 1.27 1.27)) (justify left bottom))
+  )
+  (label "A13" (at 40.64 36.83 0) (fields_autoplaced)
+    (effects (font (size 1.27 1.27)) (justify left bottom))
+  )
+  (label "A9" (at 24.13 118.11 0) (fields_autoplaced)
+    (effects (font (size 1.27 1.27)) (justify left bottom))
+  )
+  (label "A4" (at 24.13 137.16 0) (fields_autoplaced)
+    (effects (font (size 1.27 1.27)) (justify left bottom))
+  )
+  (label "A15" (at 40.64 41.91 0) (fields_autoplaced)
+    (effects (font (size 1.27 1.27)) (justify left bottom))
+  )
+  (label "A14" (at 40.64 39.37 0) (fields_autoplaced)
+    (effects (font (size 1.27 1.27)) (justify left bottom))
+  )
+  (label "A1" (at 57.15 113.03 0) (fields_autoplaced)
+    (effects (font (size 1.27 1.27)) (justify left bottom))
+  )
+  (label "A10" (at 24.13 114.3 0) (fields_autoplaced)
     (effects (font (size 1.27 1.27)) (justify left bottom))
   )
@@
     )
   )
-  (symbol (lib_id "74xx:74LS00") (at 265.43 120.65 0) (unit 2)
-    (in_bom yes) (on_board yes) (dnp no) (fields_autoplaced)
-    (property "Reference" "U10" (at 265.4217 113.03 0)
-      (effects (font (size 1.27 1.27)))
-    )
-    (property "Value" "74HCT00" (at 265.4217 115.57 0)
-      (effects (font (size 1.27 1.27)))
-    )
-    (property "Footprint" "Package_DIP:DIP-14_W7.62mm" (at 265.43 120.65 0)
-      (effects (font (size 1.27 1.27)) hide)
-    )
-    (property "Datasheet" "http://www.ti.com/lit/gpn/sn74ls00" (at 265.43 120.65 0)
-      (effects (font (size 1.27 1.27)) hide)
-    )
+  (symbol (lib_id "74xx:74LS00") (at 265.43 110.49 0) (unit 2)
+    (in_bom yes) (on_board yes) (dnp no) (fields_autoplaced)
+    (property "Reference" "U10" (at 265.4217 102.87 0)
+      (effects (font (size 1.27 1.27)))
+    )
+    (property "Value" "74HCT00" (at 265.4217 105.41 0)
+      (effects (font (size 1.27 1.27)))
+    )
+    (property "Footprint" "Package_DIP:DIP-14_W7.62mm" (at 265.43 110.49 0)
+      (effects (font (size 1.27 1.27)) hide)
+    )
+    (property "Datasheet" "http://www.ti.com/lit/gpn/sn74ls00" (at 265.43 110.49 0)
+      (effects (font (size 1.27 1.27)) hide)
+    )

Commit message: EDA work for new expansion header
Parts:
- added unit 4 of U12
- added unit 2 of U12
- added unit 3 of U12
- renumbered U11 to U12
Connections:
- net GND: now also U12.10, U12.12, U12.13, U12.4, U12.5, U12.9
- net E000: now reaches U5.7 (O7), U6.4
- net C000: now reaches U5.9 (O6), U6.1
- no-connect marks 9 -> 12
Changed lines of the file:
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@@
   (junction (at 257.81 147.32) (diameter 0) (color 0 0 0 0)
   )
+  (junction (at 257.81 107.95) (diameter 0) (color 0 0 0 0)
+  )
   (junction (at 144.78 161.29) (diameter 0) (color 0 0 0 0)
   )
@@
   (junction (at 34.29 118.11) (diameter 0) (color 0 0 0 0)
   )
+  (junction (at 257.81 76.2) (diameter 0) (color 0 0 0 0)
+  )
   (junction (at 118.11 87.63) (diameter 0) (color 0 0 0 0)
   )
@@
   (junction (at 34.29 114.3) (diameter 0) (color 0 0 0 0)
   )
+  (junction (at 257.81 81.28) (diameter 0) (color 0 0 0 0)
+  )
   (junction (at 257.81 133.35) (diameter 0) (color 0 0 0 0)
   )
@@
   (junction (at 34.29 140.97) (diameter 0) (color 0 0 0 0)
   )
+  (junction (at 257.81 67.31) (diameter 0) (color 0 0 0 0)
+  )
+  (junction (at 257.81 95.25) (diameter 0) (color 0 0 0 0)
+  )
   (junction (at 162.56 161.29) (diameter 0) (color 0 0 0 0)
   )
@@
   )
   (junction (at 20.32 99.06) (diameter 0) (color 0 0 0 0)
+  )
+  (junction (at 257.81 90.17) (diameter 0) (color 0 0 0 0)
   )
   (junction (at 118.11 82.55) (diameter 0) (color 0 0 0 0)
@@
   (no_connect (at 73.66 41.91))
   (no_connect (at 73.66 44.45))
+  (no_connect (at 273.05 78.74))
+  (no_connect (at 273.05 64.77))
   (no_connect (at 85.09 90.17))
   (no_connect (at 273.05 130.81))
   (no_connect (at 273.05 110.49))
+  (no_connect (at 273.05 92.71))
   (no_connect (at 73.66 39.37))
   (no_connect (at 273.05 140.97))
@@
     (stroke (width 0) (type default))
   )
+  (wire (pts (xy 257.81 90.17) (xy 257.81 95.25))
+    (stroke (width 0) (type default))
+  )
   (wire (pts (xy 125.73 158.75) (xy 125.73 161.29))
     (stroke (width 0) (type default))
@@
     (stroke (width 0) (type default))
   )
+  (wire (pts (xy 257.81 62.23) (xy 257.81 67.31))
+    (stroke (width 0) (type default))
+  )
   (wire (pts (xy 257.81 133.35) (xy 257.81 138.43))
     (stroke (width 0) (type default))
@@
     (stroke (width 0) (type default))
   )
+  (wire (pts (xy 257.81 76.2) (xy 257.81 81.28))
+    (stroke (width 0) (type default))
+  )
   (wire (pts (xy 60.96 171.45) (xy 60.96 161.29))
     (stroke (width 0) (type default))
@@
     (stroke (width 0) (type default))
   )
+  (wire (pts (xy 257.81 95.25) (xy 257.81 107.95))
+    (stroke (width 0) (type default))
+  )
   (bus (pts (xy 36.83 39.37) (xy 36.83 68.58))
     (stroke (width 0) (type default))
@@
     (stroke (width 0) (type default))
   )
+  (wire (pts (xy 257.81 67.31) (xy 257.81 76.2))
+    (stroke (width 0) (type default))
+  )
   (wire (pts (xy 22.86 133.35) (xy 26.67 133.35))
     (stroke (width 0) (type default))
@@
   )
   (wire (pts (xy 257.81 147.32) (xy 257.81 152.4))
+    (stroke (width 0) (type default))
+  )
+  (wire (pts (xy 257.81 81.28) (xy 257.81 90.17))
     (stroke (width 0) (type default))
   )
@@
     (effects (font (size 1.27 1.27)) (justify left bottom))
   )
+  (label "C000" (at 91.44 52.07 0) (fields_autoplaced)
+    (effects (font (size 1.27 1.27)) (justify left bottom))
+  )
   (label "A2" (at 24.13 144.78 0) (fields_autoplaced)
     (effects (font (size 1.27 1.27)) (justify left bottom))
@@
   )
   (label "A15" (at 40.64 41.91 0) (fields_autoplaced)
+    (effects (font (size 1.27 1.27)) (justify left bottom))
+  )
+  (label "E000" (at 91.44 64.77 0) (fields_autoplaced)
     (effects (font (size 1.27 1.27)) (justify left bottom))
   )
@@
   (symbol (lib_id "74xx:74LS32") (at 69.85 175.26 0) (unit 5)
     (in_bom yes) (on_board yes) (dnp no)
-    (property "Reference" "U11" (at 66.04 173.99 0)
+    (property "Reference" "U12" (at 66.04 173.99 0)
       (effects (font (size 1.27 1.27)) (justify left))
     )
@@
       (project "main-board"
         (path "/2957ffac-6a43-4af7-8ab7-5cc1dbf2f2d7/1102bb51-c389-41c1-9936-a9da336806ff"
-          (reference "U11") (unit 5)
+          (reference "U12") (unit 5)
         )
       )
@@
         (path "/2957ffac-6a43-4af7-8ab7-5cc1dbf2f2d7/1102bb51-c389-41c1-9936-a9da336806ff"
           (reference "#PWR014") (unit 1)
+        )
+      )
+    )
+  )
+  (symbol (lib_id "74xx:74LS32") (at 265.43 92.71 0) (unit 4)
+    (in_bom yes) (on_board yes) (dnp no)
+    (property "Reference" "U12" (at 261.62 85.09 0)
+      (effects (font (size 1.27 1.27)) (justify left))
+    )
+    (property "Value" "74HCT32" (at 261.62 87.63 0)
+      (effects (font (size 1.27 1.27)) (justify left))
+    )
+    (property "Footprint" "Package_DIP:DIP-14_W7.62mm" (at 265.43 92.71 0)
+      (effects (font (size 1.27 1.27)) hide)
+    )
+    (property "Datasheet" "http://www.ti.com/lit/gpn/sn74LS32" (at 265.43 92.71 0)
+      (effects (font (size 1.27 1.27)) hide)
+    )
+    (pin "1")
+    (pin "2")
+    (pin "3")
+    (pin "4")
+    (pin "5")
+    (pin "6")
+    (pin "10")
+    (pin "8")
+    (pin "9")
+    (pin "11")
+    (pin "12")
+    (pin "13")
+    (pin "14")
+    (pin "7")
+    (instances
+      (project "main-board"
+        (path "/2957ffac-6a43-4af7-8ab7-5cc1dbf2f2d7/1102bb51-c389-41c1-9936-a9da336806ff"
+          (reference "U12") (unit 4)
         )
       )
@@
     )
   )
+  (symbol (lib_id "74xx:74LS32") (at 265.43 64.77 0) (unit 2)
+    (in_bom yes) (on_board yes) (dnp no)
+    (property "Reference" "U12" (at 261.62 57.15 0)
+      (effects (font (size 1.27 1.27)) (justify left))
+    )
+    (property "Value" "74HCT32" (at 261.62 59.69 0)
+      (effects (font (size 1.27 1.27)) (justify left))
+    )
+    (property "Footprint" "Package_DIP:DIP-14_W7.62mm" (at 265.43 64.77 0)
+      (effects (font (size 1.27 1.27)) hide)
+    )
+    (property "Datasheet" "http://www.ti.com/lit/gpn/sn74LS32" (at 265.43 64.77 0)
+      (effects (font (size 1.27 1.27)) hide)
+    )
+    (pin "1")
+    (pin "2")
+    (pin "3")
+    (pin "4")
+    (pin "5")
+    (pin "6")
+    (pin "10")
+    (pin "8")
+    (pin "9")
+    (pin "11")
+    (pin "12")
+    (pin "13")
+    (pin "14")
+    (pin "7")
+    (instances
+      (project "main-board"
+        (path "/2957ffac-6a43-4af7-8ab7-5cc1dbf2f2d7/1102bb51-c389-41c1-9936-a9da336806ff"
+          (reference "U12") (unit 2)
+        )
+      )
+    )
+  )
   (symbol (lib_id "74xx:74LS00") (at 34.29 80.01 0) (unit 1)
     (in_bom yes) (on_board yes) (dnp no) (fields_autoplaced)
@@
         )
       )
+    )
+  )
+  (symbol (lib_id "74xx:74LS32") (at 265.43 78.74 0) (unit 3)
+    (in_bom yes) (on_board yes) (dnp no)
+    (property "Reference" "U12" (at 261.62 71.12 0)
+      (effects (font (size 1.27 1.27)) (justify left))
+    )
+    (property "Value" "74HCT32" (at 261.62 73.66 0)
+      (effects (font (size 1.27 1.27)) (justify left))
+    )
+    (property "Footprint" "Package_DIP:DIP-14_W7.62mm" (at 265.43 78.74 0)
+      (effects (font (size 1.27 1.27)) hide)
+    )
+    (property "Datasheet" "http://www.ti.com/lit/gpn/sn74LS32" (at 265.43 78.74 0)
+      (effects (font (size 1.27 1.27)) hide)
+    )
+    (pin "1")
+    (pin "2")
+    (pin "3")
+    (pin "4")
+    (pin "5")
+    (pin "6")
+    (pin "10")
+    (pin "8")
+    (pin "9")
+    (pin "11")
+    (pin "12")
+    (pin "13")
+    (pin "14")
+    (pin "7")
+    (instances
+      (project "main-board"
+        (path "/2957ffac-6a43-4af7-8ab7-5cc1dbf2f2d7/1102bb51-c389-41c1-9936-a9da336806ff"
+          (reference "U12") (unit 3)
+        )
+      )

Commit message: Normalize cap size
Parts:
- C3: footprint Capacitor_THT:C_Disc_D6.0mm_W2.5mm_P5.00mm -> Capacitor_THT:C_Disc_D3.8mm_W2.6mm_P2.50mm
Changed lines of the file:
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@@
       (effects (font (size 1.27 1.27)) (justify left))
     )
-    (property "Footprint" "Capacitor_THT:C_Disc_D6.0mm_W2.5mm_P5.00mm" (at 117.8052 179.07 0)
+    (property "Footprint" "Capacitor_THT:C_Disc_D3.8mm_W2.6mm_P2.50mm" (at 117.8052 179.07 0)
       (effects (font (size 1.27 1.27)) hide)
     )
@@
       (effects (font (size 1.27 1.27)) (justify left))
     )
-    (property "Footprint" "Capacitor_THT:C_Disc_D6.0mm_W2.5mm_P5.00mm" (at 39.0652 182.88 0)
+    (property "Footprint" "Capacitor_THT:C_Disc_D3.8mm_W2.6mm_P2.50mm" (at 39.0652 182.88 0)
       (effects (font (size 1.27 1.27)) hide)
     )
@@
       (effects (font (size 1.27 1.27)) (justify left))
     )
-    (property "Footprint" "Capacitor_THT:C_Disc_D6.0mm_W2.5mm_P5.00mm" (at 98.7552 179.07 0)
+    (property "Footprint" "Capacitor_THT:C_Disc_D3.8mm_W2.6mm_P2.50mm" (at 98.7552 179.07 0)
       (effects (font (size 1.27 1.27)) hide)
     )
@@
       (effects (font (size 1.27 1.27)) (justify left))
     )
-    (property "Footprint" "Capacitor_THT:C_Disc_D6.0mm_W2.5mm_P5.00mm" (at 136.8552 179.07 0)
+    (property "Footprint" "Capacitor_THT:C_Disc_D3.8mm_W2.6mm_P2.50mm" (at 136.8552 179.07 0)
       (effects (font (size 1.27 1.27)) hide)
     )
@@
       (effects (font (size 1.27 1.27)) (justify left))
     )
-    (property "Footprint" "Capacitor_THT:C_Disc_D6.0mm_W2.5mm_P5.00mm" (at 79.7052 179.07 0)
+    (property "Footprint" "Capacitor_THT:C_Disc_D3.8mm_W2.6mm_P2.50mm" (at 79.7052 179.07 0)
       (effects (font (size 1.27 1.27)) hide)
     )
@@
       (effects (font (size 1.27 1.27)) (justify left))
     )
-    (property "Footprint" "Capacitor_THT:C_Disc_D6.0mm_W2.5mm_P5.00mm" (at 154.6352 179.07 0)
+    (property "Footprint" "Capacitor_THT:C_Disc_D3.8mm_W2.6mm_P2.50mm" (at 154.6352 179.07 0)
       (effects (font (size 1.27 1.27)) hide)
     )
@@
       (effects (font (size 1.27 1.27)) (justify left))
     )
-    (property "Footprint" "Capacitor_THT:C_Disc_D6.0mm_W2.5mm_P5.00mm" (at 61.9252 179.07 0)
-      (effects (font (size 1.27 1.27)) hide)
-    )
+    (property "Footprint" "Capacitor_THT:C_Disc_D3.8mm_W2.6mm_P2.50mm" (at 61.9252 179.07 0)
+      (effects (font (size 1.27 1.27)) hide)
+    )

Commit message: Rerouting IO card
Parts:
- renumbered C3 to C10, C3 to C11, C3 to C12, C3 to C13, C3 to C14, C3 to C15, C3 to C7, R1 to R4
