File: eda/main-board/memory-banking.kicad_sch (KiCad schematic)
At the start: 7 parts, among them J2 Membank block, U14 74LHCT157, U15 74LHCT157, U16 74HCT273

Commit message: EDA work for new expansion header
Connections:
- net D0: now also U16.4 (D1); no longer U16.3 (D0)
- net D1: now also U16.3 (D0); no longer U16.4 (D1)
- net LA13: now reaches J2.2 (Pin_2), U14.2 (I0a), U16.9 (Q3)
- net LA14: now reaches J2.3 (Pin_3), U14.5 (I0b), U16.12 (Q4)
- net LA15: now reaches J2.4 (Pin_4), U14.11 (I0c), U16.15 (Q5)
- net LA17: now reaches J2.5 (Pin_5), U15.2 (I0a), U16.16 (Q6)
- net LA18: now reaches J2.6 (Pin_6), U15.5 (I0b), U16.19 (Q7)
Changed lines of the file:
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@@
+    (effects (font (size 1.27 1.27)) (justify left bottom))
+  )
+  (label "LA18" (at 133.35 113.03 0) (fields_autoplaced)
+    (effects (font (size 1.27 1.27)) (justify left bottom))
+  )
+  (label "LA15" (at 130.81 52.07 0) (fields_autoplaced)
     (effects (font (size 1.27 1.27)) (justify left bottom))
   )
@@
     (effects (font (size 1.27 1.27)) (justify left bottom))
   )
-  (label "D1" (at 57.15 71.12 0) (fields_autoplaced)
+  (label "D1" (at 57.15 68.58 0) (fields_autoplaced)
+    (effects (font (size 1.27 1.27)) (justify left bottom))
+  )
+  (label "LA14" (at 130.81 44.45 0) (fields_autoplaced)
     (effects (font (size 1.27 1.27)) (justify left bottom))
   )
@@
     (effects (font (size 1.27 1.27)) (justify left bottom))
   )
+  (label "LA17" (at 132.08 105.41 0) (fields_autoplaced)
+    (effects (font (size 1.27 1.27)) (justify left bottom))
+  )
   (label "D2" (at 57.15 73.66 0) (fields_autoplaced)
     (effects (font (size 1.27 1.27)) (justify left bottom))
@@
     (effects (font (size 1.27 1.27)) (justify left bottom))
   )
+  (label "LA13" (at 130.81 36.83 0) (fields_autoplaced)
+    (effects (font (size 1.27 1.27)) (justify left bottom))
+  )
   (label "D6" (at 57.15 83.82 0) (fields_autoplaced)
     (effects (font (size 1.27 1.27)) (justify left bottom))
   )
-  (label "D0" (at 57.15 68.58 0) (fields_autoplaced)
+  (label "D0" (at 57.15 71.12 0) (fields_autoplaced)
     (effects (font (size 1.27 1.27)) (justify left bottom))
   )
@@
           (reference "#PWR013") (unit 1)
         )
-        (path "/2957ffac-6a43-4af7-8ab7-5cc1dbf2f2d7/a1f91ce1-7954-4252-a94a-6925f1ee803e"
-          (reference "#PWR034") (unit 1)
-        )
         (path "/2957ffac-6a43-4af7-8ab7-5cc1dbf2f2d7/b7610ea3-6d9d-4a7a-bdcf-7fc9b6af9d5d"
           (reference "#PWR040") (unit 1)
@@
         (path "/2957ffac-6a43-4af7-8ab7-5cc1dbf2f2d7/1102bb51-c389-41c1-9936-a9da336806ff"
           (reference "#PWR013") (unit 1)
-        )
-        (path "/2957ffac-6a43-4af7-8ab7-5cc1dbf2f2d7/a1f91ce1-7954-4252-a94a-6925f1ee803e"
-          (reference "#PWR034") (unit 1)
         )
         (path "/2957ffac-6a43-4af7-8ab7-5cc1dbf2f2d7/b7610ea3-6d9d-4a7a-bdcf-7fc9b6af9d5d"
@@
         (path "/2957ffac-6a43-4af7-8ab7-5cc1dbf2f2d7/1102bb51-c389-41c1-9936-a9da336806ff"
           (reference "C7") (unit 1)
-        )
-        (path "/2957ffac-6a43-4af7-8ab7-5cc1dbf2f2d7/a1f91ce1-7954-4252-a94a-6925f1ee803e"
-          (reference "C8") (unit 1)
         )
         (path "/2957ffac-6a43-4af7-8ab7-5cc1dbf2f2d7/b7610ea3-6d9d-4a7a-bdcf-7fc9b6af9d5d"
@@
         (path "/2957ffac-6a43-4af7-8ab7-5cc1dbf2f2d7/1102bb51-c389-41c1-9936-a9da336806ff"
           (reference "#PWR014") (unit 1)
-        )
-        (path "/2957ffac-6a43-4af7-8ab7-5cc1dbf2f2d7/a1f91ce1-7954-4252-a94a-6925f1ee803e"
-          (reference "#PWR035") (unit 1)
         )
         (path "/2957ffac-6a43-4af7-8ab7-5cc1dbf2f2d7/b7610ea3-6d9d-4a7a-bdcf-7fc9b6af9d5d"
@@
           (reference "C7") (unit 1)
         )
-        (path "/2957ffac-6a43-4af7-8ab7-5cc1dbf2f2d7/a1f91ce1-7954-4252-a94a-6925f1ee803e"
-          (reference "C8") (unit 1)
-        )
         (path "/2957ffac-6a43-4af7-8ab7-5cc1dbf2f2d7/b7610ea3-6d9d-4a7a-bdcf-7fc9b6af9d5d"
           (reference "C16") (unit 1)
@@
         (path "/2957ffac-6a43-4af7-8ab7-5cc1dbf2f2d7/1102bb51-c389-41c1-9936-a9da336806ff"
           (reference "#PWR014") (unit 1)
-        )
-        (path "/2957ffac-6a43-4af7-8ab7-5cc1dbf2f2d7/a1f91ce1-7954-4252-a94a-6925f1ee803e"
-          (reference "#PWR035") (unit 1)
         )
         (path "/2957ffac-6a43-4af7-8ab7-5cc1dbf2f2d7/b7610ea3-6d9d-4a7a-bdcf-7fc9b6af9d5d"
@@
           (reference "C7") (unit 1)
         )
-        (path "/2957ffac-6a43-4af7-8ab7-5cc1dbf2f2d7/a1f91ce1-7954-4252-a94a-6925f1ee803e"
-          (reference "C8") (unit 1)
-        )
         (path "/2957ffac-6a43-4af7-8ab7-5cc1dbf2f2d7/b7610ea3-6d9d-4a7a-bdcf-7fc9b6af9d5d"
           (reference "C17") (unit 1)
@@
         (path "/2957ffac-6a43-4af7-8ab7-5cc1dbf2f2d7/1102bb51-c389-41c1-9936-a9da336806ff"
           (reference "#PWR013") (unit 1)
-        )
-        (path "/2957ffac-6a43-4af7-8ab7-5cc1dbf2f2d7/a1f91ce1-7954-4252-a94a-6925f1ee803e"
-          (reference "#PWR034") (unit 1)
         )
         (path "/2957ffac-6a43-4af7-8ab7-5cc1dbf2f2d7/b7610ea3-6d9d-4a7a-bdcf-7fc9b6af9d5d"
@@
           (reference "#PWR015") (unit 1)
         )
-        (path "/2957ffac-6a43-4af7-8ab7-5cc1dbf2f2d7/a1f91ce1-7954-4252-a94a-6925f1ee803e"
-          (reference "#PWR032") (unit 1)
-        )
         (path "/2957ffac-6a43-4af7-8ab7-5cc1dbf2f2d7/b7610ea3-6d9d-4a7a-bdcf-7fc9b6af9d5d"
           (reference "#PWR036") (unit 1)
@@
           (reference "#PWR016") (unit 1)
         )
-        (path "/2957ffac-6a43-4af7-8ab7-5cc1dbf2f2d7/a1f91ce1-7954-4252-a94a-6925f1ee803e"
-          (reference "#PWR033") (unit 1)
-        )
         (path "/2957ffac-6a43-4af7-8ab7-5cc1dbf2f2d7/b7610ea3-6d9d-4a7a-bdcf-7fc9b6af9d5d"
           (reference "#PWR037") (unit 1)
@@
           (reference "#PWR014") (unit 1)
         )
-        (path "/2957ffac-6a43-4af7-8ab7-5cc1dbf2f2d7/a1f91ce1-7954-4252-a94a-6925f1ee803e"
-          (reference "#PWR035") (unit 1)
-        )
-        (path "/2957ffac-6a43-4af7-8ab7-5cc1dbf2f2d7/b7610ea3-6d9d-4a7a-bdcf-7fc9b6af9d5d"
+        (path "/2957ffac-6a43-4af7-8ab7-5cc1dbf2f2d7/b7610ea3-6d9d-4a7a-bdcf-7fc9b6af9d5d"

Commit message: Normalize cap size
Parts:
- C3: footprint Capacitor_THT:C_Disc_D6.0mm_W2.5mm_P5.00mm -> Capacitor_THT:C_Disc_D3.8mm_W2.6mm_P2.50mm
Changed lines of the file:
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@@
       (effects (font (size 1.27 1.27)) (justify left))
     )
-    (property "Footprint" "Capacitor_THT:C_Disc_D6.0mm_W2.5mm_P5.00mm" (at 37.7952 184.15 0)
+    (property "Footprint" "Capacitor_THT:C_Disc_D3.8mm_W2.6mm_P2.50mm" (at 37.7952 184.15 0)
       (effects (font (size 1.27 1.27)) hide)
     )
@@
       (effects (font (size 1.27 1.27)) (justify left))
     )
-    (property "Footprint" "Capacitor_THT:C_Disc_D6.0mm_W2.5mm_P5.00mm" (at 49.2252 184.15 0)
+    (property "Footprint" "Capacitor_THT:C_Disc_D3.8mm_W2.6mm_P2.50mm" (at 49.2252 184.15 0)
       (effects (font (size 1.27 1.27)) hide)
     )
@@
       (effects (font (size 1.27 1.27)) (justify left))
     )
-    (property "Footprint" "Capacitor_THT:C_Disc_D6.0mm_W2.5mm_P5.00mm" (at 61.9252 184.15 0)
+    (property "Footprint" "Capacitor_THT:C_Disc_D3.8mm_W2.6mm_P2.50mm" (at 61.9252 184.15 0)
       (effects (font (size 1.27 1.27)) hide)
     )

Commit message: Rerouting IO card
Parts:
- renumbered C3 to C16, C3 to C17, C3 to C9
