File: eda/main-board/memory.kicad_sch (KiCad schematic)
At the start: 6 parts, among them J1 RomHighSel, U3 28C256, U4 AS6C4008-55PCN

Commit message: Normalize cap size
Parts:
- C3: footprint Capacitor_THT:C_Disc_D6.0mm_W2.5mm_P5.00mm -> Capacitor_THT:C_Disc_D3.8mm_W2.6mm_P2.50mm
Changed lines of the file:
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@@
       (effects (font (size 1.27 1.27)) (justify left))
     )
-    (property "Footprint" "Capacitor_THT:C_Disc_D6.0mm_W2.5mm_P5.00mm" (at 33.9852 184.15 0)
+    (property "Footprint" "Capacitor_THT:C_Disc_D3.8mm_W2.6mm_P2.50mm" (at 33.9852 184.15 0)
       (effects (font (size 1.27 1.27)) hide)
     )
@@
       (effects (font (size 1.27 1.27)) (justify left))
     )
-    (property "Footprint" "Capacitor_THT:C_Disc_D6.0mm_W2.5mm_P5.00mm" (at 44.1452 184.15 0)
-      (effects (font (size 1.27 1.27)) hide)
-    )
+    (property "Footprint" "Capacitor_THT:C_Disc_D3.8mm_W2.6mm_P2.50mm" (at 44.1452 184.15 0)
+      (effects (font (size 1.27 1.27)) hide)
+    )

Commit message: Rerouting IO card
Parts:
- renumbered C3 to C18, C3 to C19, R1 to R3
