File: eda/main-board/main-board.kicad_sch (KiCad schematic)
At the start: 14 parts, among them J4 $1-3 latch, J5 PWR, U1 W65C02SxP, X1 4Mhz

Commit message: fix: Issue on mainboard
Connections:
- net VCC: now also U1.38 (~{SO})
- no-connect marks 6 -> 5
Changed lines of the file:
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@@
-	)
-	(no_connect
-		(at 115.57 99.06)
 	)
 	(no_connect
@@
 		(pts
 			(xy 80.01 55.88) (xy 107.95 55.88)
+		)
+		(stroke
+			(width 0)
+			(type default)
+		)
+	)
+	(wire
+		(pts
+			(xy 96.52 99.06) (xy 115.57 99.06)
 		)
 		(stroke
@@
 					(unit 1)
 				)
+			)
+		)
+	)
+	(symbol
+		(lib_id "power:VCC")
+		(at 96.52 99.06 90)
+		(unit 1)
+		(exclude_from_sim no)
+		(in_bom yes)
+		(on_board yes)
+		(dnp no)
+		(fields_autoplaced yes)
+		(property "Reference" "#PWR072"
+			(at 100.33 99.06 0)
+			(effects
+				(font
+					(size 1.27 1.27)
+				)
+				(hide yes)
+			)
+		)
+		(property "Value" "VCC"
+			(at 92.71 99.0599 90)
+			(effects
+				(font
+					(size 1.27 1.27)
+				)
+				(justify left)
+			)
+		)
+		(property "Footprint" ""
+			(at 96.52 99.06 0)
+			(effects
+				(font
+					(size 1.27 1.27)
+				)
+				(hide yes)
+			)
+		)
+		(property "Datasheet" ""
+			(at 96.52 99.06 0)
+			(effects
+				(font
+					(size 1.27 1.27)
+				)
+				(hide yes)
+			)
+		)
+		(property "Description" ""
+			(at 96.52 99.06 0)
+			(effects
+				(font
+					(size 1.27 1.27)
+				)
+				(hide yes)
+			)
+		)
+		(pin "1"
+		)
+		(instances
+			(project "main-board"
+				(path "/2957ffac-6a43-4af7-8ab7-5cc1dbf2f2d7"
+					(reference "#PWR072")
+					(unit 1)
+				)
