File: eda/expansion-40-to-50-conversion/expansion-40-to-50-conversion.kicad_pcb (KiCad board)
At the start: 2 copper layers, 24.4 x 68.8 mm, 3 parts, among them J1 50pin, J2 40pin

Commit message: Touchups before ordering
Routing:
- net /GND: track 20.1 -> 25.0 mm
Changed lines of the file:
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@@
 			(outputformat 1)
 			(mirror no)
-			(drillshape 1)
+			(drillshape 0)
 			(scaleselection 1)
-			(outputdirectory "")
+			(outputdirectory "C:/Users/nojan/Desktop/Gerbers/expansion-converter/")
 		)
 	)
@@
 	)
 	(segment
+		(start 136.398 59.182)
+		(end 137.16 59.182)
+		(width 0.2)
+		(layer "B.Cu")
+		(net 2)
+	)
+	(segment
 		(start 125.476 83.312)
 		(end 127.254 83.312)
@@
 	)
 	(segment
+		(start 135.128 60.452)
+		(end 135.636 60.452)
+		(width 0.2)
+		(layer "B.Cu")
+		(net 2)
+	)
+	(segment
 		(start 121.539 64.389)
 		(end 121.031 64.389)
@@
 	)
 	(segment
+		(start 135.128 60.452)
+		(end 136.398 59.182)
+		(width 0.2)
+		(layer "B.Cu")
+		(net 2)
+	)
+	(segment
 		(start 122.936 62.992)
 		(end 121.92 61.976)
@@
 		(width 0.2)
 		(layer "B.Cu")
+		(net 2)
+	)
+	(segment
+		(start 135.636 60.452)
+		(end 136.906 61.722)
+		(width 0.2)
+		(layer "B.Cu")
