File: eda/io-card/sd-card.kicad_sch (KiCad schematic)
At the start: 8 parts, among them J8 SD-Card module, J9 SD_Card, U14 LM317L_TO92

Commit message: EDA work for new expansion header
Parts:
- added U12: 74HC541, Package_DIP:DIP-20_W7.62mm, symbol 74xx:74LS541
Connections:
- net +3.3V: now also U12.20 (VCC)
- net CardDetect: now also U12.6 (A4); no longer J8.2 (Pin_2), J9.10 (CARD_DETECT)
- net GND: now also U12.1 (G1), U12.10 (GND), U12.19 (G2), U12.8 (A6), U12.9 (A7)
- net SPI_CLK: now also U12.4 (A2); no longer J8.4 (Pin_4)
- net SPI_MISO: now also U12.15 (Y3); no longer J8.5 (Pin_5), J9.7 (DAT0)
- net SPI_MOSI: now also U12.3 (A1); no longer J8.6 (Pin_6)
- net WriteProtect: now also U12.7 (A5); no longer J8.7 (Pin_7), J9.11 (WRITE_PROTECT)
- net ~{CS}: now also U12.2 (A0); no longer J8.3 (Pin_3)
- net SD_CS: now reaches J9.1 (CD/DAT3)
- net SD_CS: now also J8.3 (Pin_3), U12.18 (Y0)
- net SD_SDO: now reaches J9.2 (CMD)
- net SD_SDO: now also J8.6 (Pin_6), U12.17 (Y1)
- net SD_CLK: now reaches J9.5 (CLK)
- net SD_CLK: now also J8.4 (Pin_4), U12.16 (Y2)
- new net SD_CardDetect: J8.2 (Pin_2), J9.10 (CARD_DETECT), U12.14 (Y4)
- new net SD_SDI: J8.5 (Pin_5), J9.7 (DAT0), U12.5 (A3)
- new net SD_WriteProtect: J8.7 (Pin_7), J9.11 (WRITE_PROTECT), U12.13 (Y5)
- no-connect marks 2 -> 4
Other:
- moved on the sheet: J9

Commit message: Normalize cap size
Parts:
- C4: footprint Capacitor_THT:C_Disc_D3.4mm_W2.1mm_P2.50mm -> Capacitor_THT:C_Disc_D3.8mm_W2.6mm_P2.50mm
Changed lines of the file:
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@@
       (effects (font (size 1.27 1.27)) (justify left))
     )
-    (property "Footprint" "Capacitor_THT:C_Disc_D3.4mm_W2.1mm_P2.50mm" (at 59.9948 40.64 0)
+    (property "Footprint" "Capacitor_THT:C_Disc_D3.8mm_W2.6mm_P2.50mm" (at 59.9948 40.64 0)
       (effects (font (size 1.27 1.27)) hide)
     )

Commit message: Rerouting IO card
Parts:
- renumbered C4 to C14, R1 to R6, R1 to R7
