File: eda/uart/fifo.kicad_sch (KiCad schematic)
At the start: 5 parts, among them IC1 CD74HCT40105E, IC2 CD74HCT40105E, U1 74HCT08

Commit message: Port main board schematic to kicad
Parts:
- C4: footprint Capacitor_THT:C_Rect_L7.2mm_W2.5mm_P5.00mm_FKS2_FKP2_MKS2_MKP2 -> Capacitor_THT:C_Rect_L7.2mm_W3.5mm_P5.00mm_FKS2_FKP2_MKS2_MKP2
Changed lines of the file:
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@@
         )
         (path "/11545594-d6d6-4b37-a578-fa23933d5773/58e4c198-6a2b-4c28-a1a8-589b85574c34/bcecd650-8eb4-42a7-a000-392fa6d28d65"
-          (reference "#PWR024") (unit 1)
-        )
-        (path "/11545594-d6d6-4b37-a578-fa23933d5773/c5eb56c0-461b-4cee-8fbe-1bd5aa80ac20/64001936-eb30-42b8-b9ac-6bd9af7e1ca4"
-          (reference "#PWR028") (unit 1)
+          (reference "#PWR026") (unit 1)
+        )
+        (path "/11545594-d6d6-4b37-a578-fa23933d5773/c5eb56c0-461b-4cee-8fbe-1bd5aa80ac20/64001936-eb30-42b8-b9ac-6bd9af7e1ca4"
+          (reference "#PWR030") (unit 1)
         )
       )
@@
         )
         (path "/11545594-d6d6-4b37-a578-fa23933d5773/58e4c198-6a2b-4c28-a1a8-589b85574c34/bcecd650-8eb4-42a7-a000-392fa6d28d65"
-          (reference "#PWR023") (unit 1)
-        )
-        (path "/11545594-d6d6-4b37-a578-fa23933d5773/c5eb56c0-461b-4cee-8fbe-1bd5aa80ac20/64001936-eb30-42b8-b9ac-6bd9af7e1ca4"
-          (reference "#PWR027") (unit 1)
+          (reference "#PWR025") (unit 1)
+        )
+        (path "/11545594-d6d6-4b37-a578-fa23933d5773/c5eb56c0-461b-4cee-8fbe-1bd5aa80ac20/64001936-eb30-42b8-b9ac-6bd9af7e1ca4"
+          (reference "#PWR029") (unit 1)
         )
       )
@@
       (effects (font (size 1.27 1.27)) (justify left))
     )
-    (property "Footprint" "Capacitor_THT:C_Rect_L7.2mm_W2.5mm_P5.00mm_FKS2_FKP2_MKS2_MKP2" (at 101.2952 137.16 0)
+    (property "Footprint" "Capacitor_THT:C_Rect_L7.2mm_W3.5mm_P5.00mm_FKS2_FKP2_MKS2_MKP2" (at 101.2952 137.16 0)
       (effects (font (size 1.27 1.27)) hide)
     )
@@
         )
         (path "/11545594-d6d6-4b37-a578-fa23933d5773/58e4c198-6a2b-4c28-a1a8-589b85574c34/bcecd650-8eb4-42a7-a000-392fa6d28d65"
-          (reference "C10") (unit 1)
-        )
-        (path "/11545594-d6d6-4b37-a578-fa23933d5773/c5eb56c0-461b-4cee-8fbe-1bd5aa80ac20/64001936-eb30-42b8-b9ac-6bd9af7e1ca4"
-          (reference "C12") (unit 1)
+          (reference "C11") (unit 1)
+        )
+        (path "/11545594-d6d6-4b37-a578-fa23933d5773/c5eb56c0-461b-4cee-8fbe-1bd5aa80ac20/64001936-eb30-42b8-b9ac-6bd9af7e1ca4"
+          (reference "C13") (unit 1)
         )
       )
@@
         )
         (path "/11545594-d6d6-4b37-a578-fa23933d5773/58e4c198-6a2b-4c28-a1a8-589b85574c34/bcecd650-8eb4-42a7-a000-392fa6d28d65"
-          (reference "U?") (unit 1)
-        )
-        (path "/11545594-d6d6-4b37-a578-fa23933d5773/c5eb56c0-461b-4cee-8fbe-1bd5aa80ac20/64001936-eb30-42b8-b9ac-6bd9af7e1ca4"
-          (reference "IC4") (unit 1)
+          (reference "U9") (unit 1)
+        )
+        (path "/11545594-d6d6-4b37-a578-fa23933d5773/c5eb56c0-461b-4cee-8fbe-1bd5aa80ac20/64001936-eb30-42b8-b9ac-6bd9af7e1ca4"
+          (reference "IC2") (unit 1)
         )
       )
@@
       (effects (font (size 1.27 1.27)) (justify left))
     )
-    (property "Footprint" "Capacitor_THT:C_Rect_L7.2mm_W2.5mm_P5.00mm_FKS2_FKP2_MKS2_MKP2" (at 115.2652 137.16 0)
+    (property "Footprint" "Capacitor_THT:C_Rect_L7.2mm_W3.5mm_P5.00mm_FKS2_FKP2_MKS2_MKP2" (at 115.2652 137.16 0)
       (effects (font (size 1.27 1.27)) hide)
     )
@@
         )
         (path "/11545594-d6d6-4b37-a578-fa23933d5773/58e4c198-6a2b-4c28-a1a8-589b85574c34/bcecd650-8eb4-42a7-a000-392fa6d28d65"
-          (reference "C11") (unit 1)
-        )
-        (path "/11545594-d6d6-4b37-a578-fa23933d5773/c5eb56c0-461b-4cee-8fbe-1bd5aa80ac20/64001936-eb30-42b8-b9ac-6bd9af7e1ca4"
-          (reference "C13") (unit 1)
+          (reference "C12") (unit 1)
+        )
+        (path "/11545594-d6d6-4b37-a578-fa23933d5773/c5eb56c0-461b-4cee-8fbe-1bd5aa80ac20/64001936-eb30-42b8-b9ac-6bd9af7e1ca4"
+          (reference "C14") (unit 1)
         )
       )
@@
         )
         (path "/11545594-d6d6-4b37-a578-fa23933d5773/c5eb56c0-461b-4cee-8fbe-1bd5aa80ac20/64001936-eb30-42b8-b9ac-6bd9af7e1ca4"
-          (reference "U6") (unit 3)
+          (reference "U1") (unit 3)
         )
       )
@@
         )
         (path "/11545594-d6d6-4b37-a578-fa23933d5773/58e4c198-6a2b-4c28-a1a8-589b85574c34/bcecd650-8eb4-42a7-a000-392fa6d28d65"
-          (reference "#PWR026") (unit 1)
-        )
-        (path "/11545594-d6d6-4b37-a578-fa23933d5773/c5eb56c0-461b-4cee-8fbe-1bd5aa80ac20/64001936-eb30-42b8-b9ac-6bd9af7e1ca4"
-          (reference "#PWR030") (unit 1)
+          (reference "#PWR028") (unit 1)
+        )
+        (path "/11545594-d6d6-4b37-a578-fa23933d5773/c5eb56c0-461b-4cee-8fbe-1bd5aa80ac20/64001936-eb30-42b8-b9ac-6bd9af7e1ca4"
+          (reference "#PWR032") (unit 1)
         )
       )
@@
         )
         (path "/11545594-d6d6-4b37-a578-fa23933d5773/58e4c198-6a2b-4c28-a1a8-589b85574c34/bcecd650-8eb4-42a7-a000-392fa6d28d65"
-          (reference "#PWR025") (unit 1)
-        )
-        (path "/11545594-d6d6-4b37-a578-fa23933d5773/c5eb56c0-461b-4cee-8fbe-1bd5aa80ac20/64001936-eb30-42b8-b9ac-6bd9af7e1ca4"
-          (reference "#PWR029") (unit 1)
+          (reference "#PWR027") (unit 1)
+        )
+        (path "/11545594-d6d6-4b37-a578-fa23933d5773/c5eb56c0-461b-4cee-8fbe-1bd5aa80ac20/64001936-eb30-42b8-b9ac-6bd9af7e1ca4"
+          (reference "#PWR031") (unit 1)
         )
       )
@@
         )
         (path "/11545594-d6d6-4b37-a578-fa23933d5773/58e4c198-6a2b-4c28-a1a8-589b85574c34/bcecd650-8eb4-42a7-a000-392fa6d28d65"
-          (reference "U?") (unit 1)
-        )
-        (path "/11545594-d6d6-4b37-a578-fa23933d5773/c5eb56c0-461b-4cee-8fbe-1bd5aa80ac20/64001936-eb30-42b8-b9ac-6bd9af7e1ca4"
-          (reference "IC3") (unit 1)
+          (reference "U8") (unit 1)
+        )
+        (path "/11545594-d6d6-4b37-a578-fa23933d5773/c5eb56c0-461b-4cee-8fbe-1bd5aa80ac20/64001936-eb30-42b8-b9ac-6bd9af7e1ca4"
+          (reference "IC1") (unit 1)
         )
       )
@@
         )
         (path "/11545594-d6d6-4b37-a578-fa23933d5773/c5eb56c0-461b-4cee-8fbe-1bd5aa80ac20/64001936-eb30-42b8-b9ac-6bd9af7e1ca4"
-          (reference "U6") (unit 4)
-        )
-      )
+          (reference "U1") (unit 4)
+        )
+      )

Commit message: Normalize cap size
Parts:
- C4: footprint Capacitor_THT:C_Rect_L7.2mm_W3.5mm_P5.00mm_FKS2_FKP2_MKS2_MKP2 -> Capacitor_THT:C_Disc_D3.8mm_W2.6mm_P2.50mm
Changed lines of the file:
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@@
       (effects (font (size 1.27 1.27)) (justify left))
     )
-    (property "Footprint" "Capacitor_THT:C_Rect_L7.2mm_W3.5mm_P5.00mm_FKS2_FKP2_MKS2_MKP2" (at 101.2952 137.16 0)
+    (property "Footprint" "Capacitor_THT:C_Disc_D3.8mm_W2.6mm_P2.50mm" (at 101.2952 137.16 0)
       (effects (font (size 1.27 1.27)) hide)
     )
@@
       (effects (font (size 1.27 1.27)) (justify left))
     )
-    (property "Footprint" "Capacitor_THT:C_Rect_L7.2mm_W3.5mm_P5.00mm_FKS2_FKP2_MKS2_MKP2" (at 115.2652 137.16 0)
+    (property "Footprint" "Capacitor_THT:C_Disc_D3.8mm_W2.6mm_P2.50mm" (at 115.2652 137.16 0)
       (effects (font (size 1.27 1.27)) hide)
     )

Commit message: Uart and loader work
Parts:
- renumbered C4 to C11, C4 to C12, IC1 to U8, IC2 to U9

Commit message: Add SPI
Changed lines of the file:
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@@
 (kicad_sch
-	(version 20231120)
+	(version 20250114)
 	(generator "eeschema")
-	(generator_version "8.0")
+	(generator_version "9.0")
 	(paper "A4")
 	(junction
@@
 	(label "D6"
 		(at 92.71 91.44 0)
-		(fields_autoplaced yes)
 		(effects
 			(font
@@
 	(label "D0"
 		(at 92.71 54.61 0)
-		(fields_autoplaced yes)
 		(effects
 			(font
@@
 	(label "D3"
 		(at 92.71 62.23 0)
-		(fields_autoplaced yes)
 		(effects
 			(font
@@
 	(label "Q4"
 		(at 143.51 86.36 0)
-		(fields_autoplaced yes)
 		(effects
 			(font
@@
 	(label "Q5"
 		(at 143.51 88.9 0)
-		(fields_autoplaced yes)
 		(effects
 			(font
@@
 	(label "Q6"
 		(at 143.51 91.44 0)
-		(fields_autoplaced yes)
 		(effects
 			(font
@@
 	(label "Q1"
 		(at 143.51 57.15 0)
-		(fields_autoplaced yes)
 		(effects
 			(font
@@
 	(label "Q3"
 		(at 143.51 62.23 0)
-		(fields_autoplaced yes)
 		(effects
 			(font
@@
 	(label "Q7"
 		(at 143.51 93.98 0)
-		(fields_autoplaced yes)
 		(effects
 			(font
@@
 	(label "D1"
 		(at 92.71 57.15 0)
-		(fields_autoplaced yes)
 		(effects
 			(font
@@
 	(label "D5"
 		(at 92.71 88.9 0)
-		(fields_autoplaced yes)
 		(effects
 			(font
@@
 	(label "D2"
 		(at 92.71 59.69 0)
-		(fields_autoplaced yes)
 		(effects
 			(font
@@
 	(label "D4"
 		(at 92.71 86.36 0)
-		(fields_autoplaced yes)
 		(effects
 			(font
@@
 	(label "Q0"
 		(at 143.51 54.61 0)
-		(fields_autoplaced yes)
 		(effects
 			(font
@@
 	(label "Q2"
 		(at 143.51 59.69 0)
-		(fields_autoplaced yes)
 		(effects
 			(font
@@
 	(label "D7"
 		(at 92.71 93.98 0)
-		(fields_autoplaced yes)
 		(effects
 			(font
@@
 		(shape input)
 		(at 171.45 96.52 0)
-		(fields_autoplaced yes)
 		(effects
 			(font
@@
 		(shape input)
 		(at 156.21 81.28 0)
-		(fields_autoplaced yes)
 		(effects
 			(font
@@
 		(shape output)
 		(at 63.5 38.1 180)
-		(fields_autoplaced yes)
 		(effects
 			(font
@@
 		(shape output)
 		(at 181.61 49.53 0)
-		(fields_autoplaced yes)
 		(effects
 			(font
@@
 		(shape input)
 		(at 64.77 46.99 180)
-		(fields_autoplaced yes)
 		(effects
 			(font
@@
 		(shape input)
 		(at 80.01 83.82 180)
-		(fields_autoplaced yes)
 		(effects
 			(font
@@
 		(shape output)
 		(at 181.61 40.64 0)
-		(fields_autoplaced yes)
 		(effects
 			(font
@@
 		(shape input)
 		(at 64.77 50.8 180)
-		(fields_autoplaced yes)
-		(effects
-			(font
+		(effects
+			(font
