File: eda/all-in-one-smc/address-decode.kicad_sch (KiCad schematic)
At the start: 10 parts, among them U2 4072, U3 74HCT32, U4 ATF16V8Bxx-xxPU, U5 74HCT139, U6 74HCT00

Commit message: wip
Parts:
- removed unit 2 of U6
Connections:
- no-connect marks 1 -> 0
Changed lines of the file:
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@@
 	)
 	(junction
-		(at 236.22 142.24)
-		(diameter 0)
-		(color 0 0 0 0)
-	)
-	(junction
 		(at 118.11 72.39)
 		(diameter 0)
 		(color 0 0 0 0)
 	)
-	(no_connect
-		(at 256.54 139.7)
-	)
 	(bus_entry
 		(at 36.83 34.29)
@@
 	(wire
 		(pts
-			(xy 236.22 142.24) (xy 236.22 143.51)
-		)
-		(stroke
-			(width 0)
-			(type default)
-		)
-	)
-	(wire
-		(pts
 			(xy 102.87 187.96) (xy 102.87 190.5)
 		)
@@
 	(wire
 		(pts
-			(xy 241.3 137.16) (xy 236.22 137.16)
-		)
-		(stroke
-			(width 0)
-			(type default)
-		)
-	)
-	(wire
-		(pts
 			(xy 162.56 161.29) (xy 162.56 162.56)
 		)
@@
 	(wire
 		(pts
-			(xy 236.22 142.24) (xy 241.3 142.24)
-		)
-		(stroke
-			(width 0)
-			(type default)
-		)
-	)
-	(wire
-		(pts
 			(xy 87.63 158.75) (xy 87.63 161.29)
 		)
@@
 	(wire
 		(pts
-			(xy 236.22 137.16) (xy 236.22 142.24)
-		)
-		(stroke
-			(width 0)
-			(type default)
-		)
-	)
-	(wire
-		(pts
 			(xy 50.8 87.63) (xy 59.69 87.63)
 		)
@@
 	)
 	(symbol
-		(lib_id "74xx:74LS00")
-		(at 248.92 139.7 0)
-		(unit 2)
-		(exclude_from_sim no)
-		(in_bom yes)
-		(on_board yes)
-		(dnp no)
-		(fields_autoplaced yes)
-		(property "Reference" "U6"
-			(at 248.9117 130.81 0)
-			(effects
-				(font
-					(size 1.27 1.27)
-				)
-			)
-		)
-		(property "Value" "74HCT00"
-			(at 248.9117 133.35 0)
-			(effects
-				(font
-					(size 1.27 1.27)
-				)
-			)
-		)
-		(property "Footprint" "Package_SO:SOIC-14_3.9x8.7mm_P1.27mm"
-			(at 248.92 139.7 0)
-			(effects
-				(font
-					(size 1.27 1.27)
-				)
-				(hide yes)
-			)
-		)
-		(property "Datasheet" "http://www.ti.com/lit/gpn/sn74ls00"
-			(at 248.92 139.7 0)
-			(effects
-				(font
-					(size 1.27 1.27)
-				)
-				(hide yes)
-			)
-		)
-		(property "Description" ""
-			(at 248.92 139.7 0)
-			(effects
-				(font
-					(size 1.27 1.27)
-				)
-				(hide yes)
-			)
-		)
-		(pin "1"
-		)
-		(pin "2"
-		)
-		(pin "3"
-		)
-		(pin "4"
-		)
-		(pin "5"
-		)
-		(pin "6"
-		)
-		(pin "10"
-		)
-		(pin "8"
-		)
-		(pin "9"
-		)
-		(pin "11"
-		)
-		(pin "12"
-		)
-		(pin "13"
-		)
-		(pin "14"
-		)
-		(pin "7"
-		)
-		(instances
-			(project "all-in-one-smc"
-				(path "/2957ffac-6a43-4af7-8ab7-5cc1dbf2f2d7/1102bb51-c389-41c1-9936-a9da336806ff"
-					(reference "U6")
-					(unit 2)
-				)
-			)
-		)
-	)
-	(symbol
 		(lib_id "power:VCC")
 		(at 102.87 158.75 0)
@@
 					(unit 1)
 				)
-			)
-		)
-	)
-	(symbol
-		(lib_id "power:GND")
-		(at 236.22 143.51 0)
-		(unit 1)
-		(exclude_from_sim no)
-		(in_bom yes)
-		(on_board yes)
-		(dnp no)
-		(fields_autoplaced yes)
-		(property "Reference" "#PWR093"
-			(at 236.22 149.86 0)
-			(effects
-				(font
-					(size 1.27 1.27)
-				)
-				(hide yes)
-			)
-		)
-		(property "Value" "GND"
-			(at 236.22 148.59 0)
-			(effects
-				(font
-					(size 1.27 1.27)
-				)
-			)
-		)
-		(property "Footprint" ""
-			(at 236.22 143.51 0)
-			(effects
-				(font
-					(size 1.27 1.27)
-				)
-				(hide yes)
-			)
-		)
-		(property "Datasheet" ""
-			(at 236.22 143.51 0)
-			(effects
-				(font
-					(size 1.27 1.27)
-				)
-				(hide yes)
-			)
-		)
-		(property "Description" ""
-			(at 236.22 143.51 0)
-			(effects
-				(font
-					(size 1.27 1.27)
-				)
-				(hide yes)
-			)
-		)
-		(pin "1"
-		)
-		(instances
-			(project "all-in-one-smc"
-				(path "/2957ffac-6a43-4af7-8ab7-5cc1dbf2f2d7/1102bb51-c389-41c1-9936-a9da336806ff"
-					(reference "#PWR093")
-					(unit 1)
-				)
