File: eda/all-in-one-smc/all-in-one-smc.kicad_sch (KiCad schematic)
At the start: 13 parts, among them J1 Audio out, J2 PWR, J3 $1-3 latch, U1 W65C02SxP, X1 4Mhz

Commit message: wip
Parts:
- removed J1: Audio out, Connector_PinHeader_2.54mm:PinHeader_1x03_P2.54mm_Vertical, symbol Connector:Conn_01x03_Pin
- removed J2: PWR, Connector_BarrelJack:BarrelJack_Horizontal, symbol Connector:Screw_Terminal_01x02
- added J2: PWR_Switch, Connector_PinHeader_2.54mm:PinHeader_1x02_P2.54mm_Vertical, symbol Connector:Conn_01x02_Pin
- added J8: USB_C PWR, Connector_USB:USB_C_Receptacle_GCT_USB4105-xx-A_16P_TopMnt_Horizontal, symbol Connector:USB_C_Receptacle_USB2.0_14P
- added R17, R18: 5.1k, Resistor_SMD:R_0805_2012Metric, symbol Device:R
Connections:
- net GND: now also J8.A1 (GND), J8.A12 (GND), J8.B1 (GND), J8.B12 (GND), J8.S1 (SHIELD), R17.2, R18.2
- net VCC: now also J2.2 (Pin_2)
- new net: J2.1 (Pin_1), J8.A4 (VBUS), J8.A9 (VBUS), J8.B4 (VBUS), J8.B9 (VBUS)
- new net: J8.A5 (CC1), R18.1
- new net: J8.B5 (CC2), R17.1
- no-connect marks 6 -> 10
Other:
- moved on the sheet: C2, D1, H1, H2, H3, H4, R1
