File: eda/all-in-one-smc/gpu.kicad_sch (KiCad schematic)
At the start: 39 parts, among them J7 ProgrammingConnector, J8 VGA, Q1 2N7002, SW1 BOOT, SW2 RST, U16 W25Q128JVS, U19 RP2040, U21 SN74LVC245APW, U22 SN74LVC245APW, Y2 ABM8-272-T3

Commit message: wip
Parts:
- removed J8: VGA, Connector_Dsub:DSUB-15-HD_Pins_Horizontal_P2.29x1.90mm_EdgePinOffset3.03mm_Housed_MountingHolesOffset4.94mm, symbol Connector:DE15_Pins_HighDensity_MountingHoles
- removed R17: 47, Resistor_SMD:R_0805_2012Metric, symbol Device:R
- removed R18, R21, R24: 500, Resistor_SMD:R_0805_2012Metric, symbol Device:R
- removed R19, R22: 1k, Resistor_SMD:R_0805_2012Metric, symbol Device:R
- removed R20, R23: 2k, Resistor_SMD:R_0805_2012Metric, symbol Device:R
- added J1: Audio out, Connector_PinHeader_2.54mm:PinHeader_1x03_P2.54mm_Vertical, symbol Connector:Conn_01x03_Pin
- added J14: HDMI_A, Connector_Video:HDMI_A_Molex_208658-1001_Horizontal, symbol Connector:HDMI_A
- added R43: 2k2, Resistor_SMD:R_0805_2012Metric, symbol Device:R
- added RN1: 270, Resistor_SMD:R_Array_Convex_8x0602, symbol Device:R_Pack08
- R16: value 47 -> 270
- R25: value 1k -> 2k2
- R26: value 2k -> 2k2
Connections:
- net +3.3V: now also R25.2
- net GND: now also J14.11 (CKS), J14.17 (GND), J14.2 (D2S), J14.5 (D1S), J14.8 (D0S), J14.SH
- net DVI_CEC: now reaches R25.1
- net DVI_CEC: now also R16.1, U19.37 (GPIO25); no longer U19.36 (GPIO24)
- net DVI_CK+: now reaches U19.27 (GPIO16)
- net DVI_CK+: now also RN1.7 (R7.1)
- net DVI_D1+: now reaches U19.31 (GPIO20)
- net DVI_D1+: now also RN1.3 (R3.1)
- net DVI_SDA: now reaches U19.35 (GPIO23)
- net DVI_SDA: now also J14.16 (SDA), R43.1
- net DVI_CK-: now reaches U19.18 (GPIO15)
- net DVI_CK-: now also RN1.8 (R8.1); no longer R16.1
- net DVI_D2-: now reaches U19.32 (GPIO21)
- net DVI_D2-: now also RN1.2 (R2.1)
- net DVI_D0+: now reaches U19.29 (GPIO18)
- net DVI_D0+: now also RN1.5 (R5.1)
- net DVI_SCL: now reaches R26.1
- net DVI_SCL: now also U19.36 (GPIO24), J14.15 (SCL); no longer U19.37 (GPIO25)
- net DVI_D0-: now reaches U19.28 (GPIO17)
- net DVI_D0-: now also RN1.6 (R6.1)
- net DVI_D1-: now reaches U19.30 (GPIO19)
- net DVI_D1-: now also RN1.4 (R4.1)
- net DVI_D2+: now reaches U19.34 (GPIO22)
- net DVI_D2+: now also RN1.1 (R1.1)
- net VGA_B renamed VCC
- net VCC: now also J14.18 (+5V), R43.2; no longer R25.2
- net VGA_Hsync: no longer names the net of R16.2
- net VGA_Hsync: now also J14.13 (CEC)
- new net: J14.1 (D2+), RN1.16 (R1.2)
- new net: J14.10 (CK+), RN1.10 (R7.2)
- new net: J14.12 (CK-), RN1.9 (R8.2)
- new net: J14.3 (D2-), RN1.15 (R2.2)
- new net: J14.4 (D1+), RN1.14 (R3.2)
- new net: J14.6 (D1-), RN1.13 (R4.2)
- new net: J14.7 (D0+), RN1.12 (R5.2)
- new net: J14.9 (D0-), RN1.11 (R6.2)
- no-connect marks 7 -> 4
Other:
- moved on the sheet: C22, C26, Q1, R15
