File: eda/all-in-one-smc/io-card.kicad_sch (KiCad schematic)
At the start: 8 parts, among them J9 VIA Breakout, U18 W65C22SxP, U20 W65C22SxP, U23 74HCT14

Commit message: wip
Parts:
- removed JP1: IRQ Select, Connector_PinHeader_2.54mm:PinHeader_1x03_P2.54mm_Vertical, symbol Jumper:Jumper_3_Open
- added U6: 74HCT00, Package_SO:SOIC-14_3.9x8.7mm_P1.27mm, symbol 74xx:74LS00
Connections:
- net GND: now also J9.24 (Pin_24)
- net ~{IRQ}: now also J9.26 (Pin_26)
- net ~{NMI}: now also J9.30 (Pin_30)
- net ~{SPI_CS2}: now also U6.4, U6.5
- net ~{UserViaIRQ}: now reaches U18.21 (~{IRQ})
- net ~{UserViaIRQ}: now also J9.28 (Pin_28)
- new net Clock/CS: U6.6
Other:
- added sheet Clock (clock.kicad_sch)
