File: eda/all-in-one-smc/ps2-keyboard-interface.kicad_sch (KiCad schematic)
At the start: 11 parts, among them J10 PS2, U23 74HCT14, U29 74HCT595, U30 74HCT595

Commit message: Working on new SPI support
Parts:
- removed JP2: Enable PS2 Output, Connector_PinHeader_2.54mm:PinHeader_1x02_P2.54mm_Vertical, symbol Jumper:Jumper_2_Open
- removed R28: 10k, Resistor_SMD:R_0805_2012Metric, symbol Device:R
Connections:
- net ~{KeyboardOut_Enable}: now also U30.13 (~{OE})
- net ~{PS2ShiftOE}: no longer U30.13 (~{OE})
- net KeyboardBit7 renamed DIO7
Other:
- moved on the sheet: U30
