File: eda/all-in-one-smc/serial.kicad_sch (KiCad schematic)
At the start: 9 parts, among them P1 USB_C_Plug_USB2.0, U14 W65C51NxQ, U15 CH340K, Y1 1.8432Mhz

Commit message: wip
Parts:
- removed P1: USB_C_Plug_USB2.0, Connector_USB:USB_C_Receptacle_GCT_USB4105-xx-A_16P_TopMnt_Horizontal, symbol Connector:USB_C_Plug_USB2.0
- added J15: USB_C Serial, Connector_USB:USB_C_Receptacle_GCT_USB4105-xx-A_16P_TopMnt_Horizontal, symbol Connector:USB_C_Receptacle_USB2.0_14P
Connections:
- net GND: now also J15.A1 (GND), J15.A12 (GND), J15.B1 (GND), J15.B12 (GND), J15.S1 (SHIELD)
- net at U15.1 (UD+): now also J15.A6 (D+), J15.B6 (D+)
- net at U15.2 (UD-): now also J15.A7 (D-), J15.B7 (D-)
- new net: J15.A4 (VBUS), J15.A9 (VBUS), J15.B4 (VBUS), J15.B9 (VBUS)
Changed lines of the file:
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@@
+	)
+	(junction
+		(at 175.26 82.55)
+		(diameter 0)
+		(color 0 0 0 0)
 	)
 	(junction
@@
 	)
 	(junction
+		(at 175.26 77.47)
+		(diameter 0)
+		(color 0 0 0 0)
+	)
+	(junction
 		(at 127 30.48)
 		(diameter 0)
@@
 	(wire
 		(pts
+			(xy 176.53 80.01) (xy 175.26 80.01)
+		)
+		(stroke
+			(width 0)
+			(type default)
+		)
+	)
+	(wire
+		(pts
 			(xy 133.35 86.36) (xy 121.92 86.36)
 		)
@@
 	(wire
 		(pts
+			(xy 175.26 80.01) (xy 175.26 77.47)
+		)
+		(stroke
+			(width 0)
+			(type default)
+		)
+	)
+	(wire
+		(pts
 			(xy 88.9 73.66) (xy 91.44 73.66)
 		)
@@
 	(wire
 		(pts
-			(xy 176.53 82.55) (xy 171.45 82.55)
+			(xy 176.53 82.55) (xy 175.26 82.55)
 		)
 		(stroke
@@
 	(wire
 		(pts
-			(xy 176.53 77.47) (xy 170.18 77.47)
+			(xy 176.53 77.47) (xy 175.26 77.47)
 		)
 		(stroke
@@
 	(wire
 		(pts
+			(xy 175.26 82.55) (xy 175.26 85.09)
+		)
+		(stroke
+			(width 0)
+			(type default)
+		)
+	)
+	(wire
+		(pts
 			(xy 88.9 63.5) (xy 88.9 38.1)
 		)
@@
 	(wire
 		(pts
+			(xy 175.26 77.47) (xy 170.18 77.47)
+		)
+		(stroke
+			(width 0)
+			(type default)
+		)
+	)
+	(wire
+		(pts
 			(xy 104.14 115.57) (xy 104.14 118.11)
 		)
@@
 		)
 	)
+	(wire
+		(pts
+			(xy 175.26 82.55) (xy 171.45 82.55)
+		)
+		(stroke
+			(width 0)
+			(type default)
+		)
+	)
 	(bus
 		(pts
@@
 		(pts
 			(xy 88.9 93.98) (xy 91.44 93.98)
+		)
+		(stroke
+			(width 0)
+			(type default)
+		)
+	)
+	(wire
+		(pts
+			(xy 175.26 85.09) (xy 176.53 85.09)
 		)
 		(stroke
@@
 				(path "/2957ffac-6a43-4af7-8ab7-5cc1dbf2f2d7/13a62835-3c16-44b1-a0dd-ab885c2e0f44"
 					(reference "#PWR057")
+					(unit 1)
+				)
+			)
+		)
+	)
+	(symbol
+		(lib_id "Connector:USB_C_Receptacle_USB2.0_14P")
+		(at 191.77 80.01 0)
+		(mirror y)
+		(unit 1)
+		(exclude_from_sim no)
+		(in_bom yes)
+		(on_board yes)
+		(dnp no)
+		(property "Reference" "J15"
+			(at 191.77 57.15 0)
+			(effects
+				(font
+					(size 1.27 1.27)
+				)
+			)
+		)
+		(property "Value" "USB_C Serial"
+			(at 191.77 59.69 0)
+			(effects
+				(font
+					(size 1.27 1.27)
+				)
+			)
+		)
+		(property "Footprint" "Connector_USB:USB_C_Receptacle_GCT_USB4105-xx-A_16P_TopMnt_Horizontal"
+			(at 187.96 80.01 0)
+			(effects
+				(font
+					(size 1.27 1.27)
+				)
+				(hide yes)
+			)
+		)
+		(property "Datasheet" "https://www.usb.org/sites/default/files/documents/usb_type-c.zip"
+			(at 187.96 80.01 0)
+			(effects
+				(font
+					(size 1.27 1.27)
+				)
+				(hide yes)
+			)
+		)
+		(property "Description" "USB 2.0-only 14P Type-C Receptacle connector"
+			(at 191.77 80.01 0)
+			(effects
+				(font
+					(size 1.27 1.27)
+				)
+				(hide yes)
+			)
+		)
+		(pin "S1"
+		)
+		(pin "A12"
+		)
+		(pin "A1"
+		)
+		(pin "A9"
+		)
+		(pin "A4"
+		)
+		(pin "B1"
+		)
+		(pin "B12"
+		)
+		(pin "B4"
+		)
+		(pin "B9"
+		)
+		(pin "A5"
+		)
+		(pin "B5"
+		)
+		(pin "A7"
+		)
+		(pin "B7"
+		)
+		(pin "A6"
+		)
+		(pin "B6"
+		)
+		(instances
+			(project "all-in-one-smc"
+				(path "/2957ffac-6a43-4af7-8ab7-5cc1dbf2f2d7/13a62835-3c16-44b1-a0dd-ab885c2e0f44"
+					(reference "J15")
 					(unit 1)
 				)
@@
 					(unit 1)
 				)
-			)
-		)
-	)
-	(symbol
-		(lib_id "Connector:USB_C_Plug_USB2.0")
-		(at 191.77 80.01 0)
-		(mirror y)
-		(unit 1)
-		(exclude_from_sim no)
-		(in_bom yes)
-		(on_board yes)
-		(dnp no)
-		(fields_autoplaced yes)
-		(property "Reference" "P1"
-			(at 203.2 78.7399 0)
-			(effects
-				(font
-					(size 1.27 1.27)
-				)
-				(justify right)
-			)
-		)
-		(property "Value" "USB_C_Plug_USB2.0"
-			(at 203.2 81.2799 0)
-			(effects
-				(font
-					(size 1.27 1.27)
-				)
-				(justify right)
-			)
-		)
-		(property "Footprint" "Connector_USB:USB_C_Receptacle_GCT_USB4105-xx-A_16P_TopMnt_Horizontal"
-			(at 187.96 80.01 0)
-			(effects
-				(font
-					(size 1.27 1.27)
-				)
-				(hide yes)
-			)
-		)
-		(property "Datasheet" "https://www.usb.org/sites/default/files/documents/usb_type-c.zip"
-			(at 187.96 80.01 0)
-			(effects
-				(font
-					(size 1.27 1.27)
-				)
-				(hide yes)
-			)
-		)
-		(property "Description" "USB 2.0-only Type-C Plug connector"
-			(at 191.77 80.01 0)
-			(effects
-				(font
-					(size 1.27 1.27)
-				)
-				(hide yes)
-			)
-		)
-		(pin "A6"
-		)
-		(pin "B9"
-		)
-		(pin "B12"
-		)
-		(pin "B1"
-		)
-		(pin "A4"
-		)
-		(pin "B5"
-		)
-		(pin "A5"
-		)
-		(pin "A12"
-		)
-		(pin "B4"
-		)
-		(pin "A9"
-		)
-		(pin "A7"
-		)
-		(pin "A1"
-		)
-		(pin "S1"
-		)
-		(instances
-			(project ""
-				(path "/2957ffac-6a43-4af7-8ab7-5cc1dbf2f2d7/13a62835-3c16-44b1-a0dd-ab885c2e0f44"
-					(reference "P1")
-					(unit 1)
-				)
